File: revB/cad/eagle/warp-revB.brd (EAGLE design)
At the start: 48 x 74.3 mm, 180 parts, among them J1 CORTEX_DEBUG_SMD, J2 DF40FC-20DP-0.4V(51), J3 DF40FC-20DP-0.4V(51), J4 DF40FC-20DP-0.4V(51)SOCKET, J5 DF40FC-20DP-0.4V(51)SOCKET, J6 QIIC connector, J7 ZX62-AB-5PA(31)MICRO-AB-SMT, U1 ADXL362, U10 TCS34725FN, U11 GRIDEYE, U12 PAN1326C, U13 SI4705, U14 TS5A3154, U15 MKL03Z32CAF4RQFN24, U16 LPS25H, U17 CCS811, U18 FT4222H, U19 TPS82740B, U2 BME680LGA, U20 ISL23415UTQFN, U21 BQ25570PVQFN, U22 SERIAL-NOR-FLASHWSON-6X5, U23 ISL23415UTQFN, U24 ICE40UP5K-SG48QFN48, U25 TLV757P, U3 BMX055, U4 HDC1000, U5 L3GD20H, U6 TPS82740A, U7 MAG3110, U8 MMA8451Q, U9 SI7021, Y1 CM519-SMD, Y2 CS325

Commit message: solved power issues and added RV8803 support
Parts:
- removed C1, C2, C4, C5, C6, C7, C8, C9: XH414HGIV01E, XH414HGIV01E:XH414HGIV01E
- removed C10, C12, C14, C16, C18, C20, C21, C23, C26, C28, C3, C32, C34, C37, C38, C46, C48, C51, C52, C53, C54, C56, C58, C60, C66, C70, C73, C75, C78, C81: 0.1uF, SparkFun-Passives:0402-CAP
- removed C11, C13, C17, C22, C27, C29, C39, C47, C67, C68, C69, C74, C77, C80: 1uF, SparkFun-Passives:0402-CAP
- removed C15, C30, C33, C72: 10uF, SparkFun-Passives:0402-CAP
- removed C19, C42, C44, C50: 4.7uF, SparkFun-Passives:0402-CAP
- removed C24: 10nF (25V), SparkFun-Passives:0402-CAP
- removed C25, C31: 33pF, SparkFun-Passives:0402-CAP
- removed C35: 22nF, SparkFun-Passives:0402-CAP
- removed C36, C55, C57, C59, C61: 4.7uF (pol), SparkFun-Passives:0402-CAP
- removed C40: 2.2uF, SparkFun-Passives:0402-CAP
- removed C41: 1.0uF, SparkFun-Passives:0402-CAP
- removed C43: 0.01uF, SparkFun-Passives:0402-CAP
- removed C45, C71, C76, C79, C82: 10nF, SparkFun-Passives:0402-CAP
- removed C49: 22uF, SparkFun-Passives:0603-CAP
- removed C62: 0.47uF, SparkFun-Passives:0402-CAP
- removed C63: 100pF, SparkFun-Passives:0402-CAP
- removed C64, C65: 27pF, SparkFun-Passives:0402-CAP
- removed D1: KXOB22-04X3F, KX0B22-04X3F:KXOB22-04X3F
- removed FB1: 600R/1A, SparkFun-Passives:0603
- removed J6: QIIC connector, SparkX:1X04_1MM_RA
- removed J7: ZX62-AB-5PA(31)MICRO-AB-SMT, ZX62-AB-5PA(31):ZX62-AB-5PA(31)
- removed L2: 10uH, PowerMagnetics (rev17f):WE-TPC_2811/2813_OLD
- removed L3: 22uH, PowerMagnetics (rev17f):WE-TPC_3816
- removed LED1, LED2, LED3, LED4: (no value), led:SML0603
- removed R1, R2, R3, R41: 4.7k, SparkFun-Passives:0402-RES
- removed R10: 4.7K, SparkFun-Passives:0402-RES
- removed R11: 10K, SparkFun-Passives:0402-RES
- removed R12, R40, R43: 10k, SparkFun-Passives:0402-RES
- removed R13, R14, R15, R23, R8: 10k, SparkFun-Resistors:0402
- removed R16: 7.32M, SparkFun-Passives:0402-RES
- removed R17: 1.91M, SparkFun-Passives:0402-RES
- removed R18, R20: 5.62M, SparkFun-Passives:0402-RES
- removed R19: 5.49M, SparkFun-Passives:0402-RES
- removed R21: 4.22M, SparkFun-Passives:0402-RES
- removed R22: 8.66M, SparkFun-Passives:0402-RES
- removed R24, R26, R28, R29, R30, R31, R32, R33, R34, R35, R36, R37, R38, R39: 0, SparkFun-Resistors:0402
- removed R25: 1M, SparkFun-Resistors:0402
- removed R27, R7: 0, SparkFun-Passives:0402-RES
- removed R4: 20, SparkFun-Resistors:0402
- removed R42, R6: DNP, SparkFun-Passives:0402-RES
- removed R5: 47k, SparkFun-Resistors:0402
- removed R9: 12k (1%), SparkFun-Resistors:0402
- removed S3: EVPAYG0BAEVPAYG0BA, EVPAYG0BA:EVPAYG0BA
- removed S4: CHS04SLIDESWITCHA-PKG-VARIANT, CHS04SLIDESWITCH:CHS04SLIDESWITCH
- removed TP19, TP20, TP21: TPTP06R, testpad:TP06R
- removed TP25: TPSTP06R, testpad:TP06R
- removed U1: ADXL362, ADXL362:ADXL362
- removed U10: TCS34725FN, TCS3772:TCS3772
- removed U11: GRIDEYE, Grideye:GRIDEYE-AMG88
- removed U12: PAN1326C, PAN1326B:PAN1326B
- removed U13: SI4705, SI4705:SI4705
- removed U14: TS5A3154, TS5A3154:TS5A3154
- removed U15: MKL03Z32CAF4RQFN24, MKL03Z32CAF4R:MKL03Z32VFK4R
- removed U16: LPS25H, LPS25H:LPS25H
- removed U17: CCS811, SparkFun-Sensors:LGA10
- removed U18: FT4222H, FT4222H:FT4222H
- removed U19: TPS82740B, TPS82740:TPS82740
- removed U2: BME680LGA, BME680:BME680
- removed U20, U23: ISL23415UTQFN, ISL23415:ISL23415
- removed U21: BQ25570PVQFN, BQ25570:BQ25570
- removed U22: SERIAL-NOR-FLASHWSON-6X5, WSON-6x5:WSON-6X5
- removed U24: ICE40UP5K-SG48QFN48, Lattice-QFN48:LATTICE-QFN-48
- removed U25: TLV757P, TLV757P:TLV757P-WSON
- removed U3: BMX055, BMX055:BMX055
- removed U4: HDC1000, HDC1000:HDC1000
- removed U5: L3GD20H, L3GD20H:L3GD20H
- removed U6: TPS82740A, TPS82740:TPS82740
- removed U7: MAG3110, MAG3110:MAG3110
- removed U8: MMA8451Q, MMA8451Q:MMA8451Q
- removed U9: SI7021, SI7021:SI7021
- removed Y1: CM519-SMD, CM519:CM519
- removed Y2: CS325, CS325:CS325
- added BOOST:C1, BOOST:C2, BOOST:C4, BOOST:C5, BOOST:C6, BOOST:C7, BOOST:C8, BOOST:C9: CPX3225A7552D, CPX3225A752D:CPX3225A752D
- added BOOST:C42, BOOST:C44, CHARGER:C2, CHARGER:C3, FPGA:C2, FT4222:C1: 4.7uF, SparkFun-Passives:0805
- added BOOST:C43, FPGA:C10, FPGA:C11, FPGA:C12, FPGA:C6, FT4222:C2, RTC:C1: 0.1uF, SparkFun-Passives:0603-CAP
- added BOOST:C45: 10nF, SparkFun-Passives:0603-CAP
- added BOOST:C49: 22uF, SparkFun-Passives:0805
- added BOOST:L2: 22uH, EMCComponents (rev19c):WE-TPC_3816
- added BOOST:L3: 10uH, EMCComponents (rev19c):WE-TPC_2811/2813_OLD
- added BOOST:R16: 4.02M, SparkFun-Passives:0402-RES
- added BOOST:R17: 1.3M, SparkFun-Passives:0402-RES
- added BOOST:R18: 6.49M, SparkFun-Passives:0402-RES
- added BOOST:R19: 5.36M, SparkFun-Passives:0402-RES
- added BOOST:R20: 9.09M, SparkFun-Passives:0402-RES
- added BOOST:R21: 8.87M, SparkFun-Passives:0402-RES
- added BOOST:R22: 4.22M, SparkFun-Passives:0402-RES
- added BOOST:TP1, BOOST:TP2, BOOST:TP3, BOOST:TP4, CHARGER:TP1, CHARGER:TP2, FPGA:TP11, MPU:TP25, RTC:TP12, USB:TP1: TPSTP06R, testpad:TP06R
- added BOOST:U21: BQ25570PVQFN, BQ25570:BQ25570
- added CHARGER:C1, FPGA:C13, FPGA:C14, FPGA:C3: 1uF, SparkFun-Passives:0805
- added CHARGER:D1, CHARGER:D2: (no value), SparkFun-LED:LED-0603
- added CHARGER:R1: 2.94k, SparkFun-Passives:0402-RES
- added CHARGER:R2: 4.32k, SparkFun-Passives:0402-RES
- added CHARGER:R3, FPGA:R43, MPU:R11, MPU:R12, MPU:R7, RTC:R40, RTC:R6: 10k, SparkFun-Passives:0402-RES
- added CHARGER:R4, CHARGER:R5, FPGA:R41, MPU:R10: 4.7k, SparkFun-Passives:0402-RES
- added CHARGER:R6: 56.2k, SparkFun-Passives:0402-RES
- added CHARGER:U$1: BQ24230VQFN, BQ24230:PVQFN-N16
- added DF40_SOCKETS:J1, DF40_SOCKETS:J2: DF40FC-20DP-0.4V(51)SOCKET, DF40C-20DS-0.4V(51):DF40C-20DP-0.4V(51)
- added FPGA:C4, FPGA:C76, FPGA:C79: 10nF, SparkFun-Passives:0402-CAP
- added FPGA:C5, REG:C1, REG:C2: 10uF, SparkFun-Passives:0805
- added FPGA:D1: BLUE, SparkFun-LED:LED-0603
- added FPGA:L1: 2.2uH, WURTH-744025002:WURTH-744025002
- added FPGA:R27: 100, SparkFun-Passives:0402-RES
- added FPGA:R42: DNP, SparkFun-Passives:0402-RES
- added FPGA:U$1: TPS62746DSBGA(8), TPS62746:DSBGA
- added FPGA:U$7: ICE40UP5K-UWG30, ICE40UP5K:LATTICE-WLCSP-30
- added FT4222:C62: 0.47uF, SparkFun-Passives:0402-CAP
- added FT4222:C63: 100pF, SparkFun-Passives:0402-CAP
- added FT4222:C64, FT4222:C65: 27pF, SparkFun-Passives:0402-CAP
- added FT4222:R23, FT4222:R25, FT4222:R5, FT4222:R8, FT4222:R9, SENSORS-1:R4: (no value), SparkFun-Resistors:0402
- added FT4222:U18: FT4222H, FT4222H:FT4222H
- added FT4222:Y2: CS325, CS325:CS325
- added MPU:C25, MPU:C31: 33pF, SparkFun-Passives:0402-CAP
- added MPU:C36, USB:C61: 4.7uF (pol), SparkFun-Passives:0402-CAP
- added MPU:C37, MPU:C51, RF:C32, RF:C34, SENSORS-1:C10, SENSORS-1:C12, SENSORS-1:C26, SENSORS-1:C28, SENSORS-1:C3, SENSORS-1:C52, SENSORS-1:C53, SENSORS-2:C14, SENSORS-2:C16, SENSORS-2:C18, SENSORS-2:C20, SENSORS-2:C21, SENSORS-2:C23, SENSORS-2:C38, SENSORS-2:C46, SENSORS-2:C48, USB:C66: 0.1uF, SparkFun-Passives:0402-CAP
- added MPU:J1: CORTEX_DEBUG_SMD, SparkFun-Connectors:SAMTECH_FTSH-105-01
- added MPU:S3: EVPAYG0BAEVPAYG0BA, EVPAYG0BA:EVPAYG0BA
- added MPU:U$1: AT45DB641E, AT45D_Flash:UDFN
- added MPU:U1: MKL03Z32VFK4RQFN24, MKL03Z32VFK4R:MKL03Z32VFK4R
- added MPU:Y1: CM519-SMD, CM519:CM519
- added REG:L2: (no value), EMCComponents (rev19c):WE-TPC_2828_OLD
- added REG:R14, REG:R15, REG:R44, REG:R45, REG:R46: 2M, SparkFun-Passives:0402-RES
- added REG:U1: TPS6274XWSON, TPS6274x:WSON-12
- added RF:C33, SENSORS-1:C30, SENSORS-2:C15: 10uF, SparkFun-Passives:0402-CAP
- added RF:C35: 22nF, SparkFun-Passives:0402-CAP
- added RF:TP1, RF:TP19, RF:TP2, RF:TP20, RF:TP21: TPTP06R, testpad:TP06R
- added RF:U12: PAN1326C, PAN1326B:PAN1326B
- added RF:U13: SI4705, SI4705:SI4705
- added RTC:D2: 250mA/100V, SparkFun-DiscreteSemi:SOD-323
- added RTC:D3: BAS70-05, diode:SOT23
- added RTC:U$5: RV-8803-C7_RTC, Micro Crystal RTC:RV-C7
- added RTC:U$6: ML414_BATTERY_CONTACT, ML414:ML414
- added SENSORS-1:C11, SENSORS-1:C13, SENSORS-1:C27, SENSORS-1:C29, SENSORS-2:C17, SENSORS-2:C22, SENSORS-2:C39, SENSORS-2:C47: 1uF, SparkFun-Passives:0402-CAP
- added SENSORS-1:C40: 2.2uF, SparkFun-Passives:0402-CAP
- added SENSORS-1:C41: 1.0uF, SparkFun-Passives:0402-CAP
- added SENSORS-1:C50, SENSORS-2:C19: 4.7uF, SparkFun-Passives:0402-CAP
- added SENSORS-1:U1: ADXL362, ADXL362:ADXL362
- added SENSORS-1:U10: TCS34725FN, TCS3772:TCS3772
- added SENSORS-1:U11: GRIDEYE, Grideye:GRIDEYE-AMG88
- added SENSORS-1:U17: CCS811, SparkFun-Sensors:LGA10
- added SENSORS-1:U2: BME680LGA, BME680:BME680
- added SENSORS-1:U20, SENSORS-1:U23: ISL23415UTQFN, ISL23415:ISL23415
- added SENSORS-1:U3: BMX055, BMX055:BMX055
- added SENSORS-2:C24: 10nF (25V), SparkFun-Passives:0402-CAP
- added SENSORS-2:U16: LPS25H, LPS25H:LPS25H
- added SENSORS-2:U4: HDC1000, HDC1000:HDC1000
- added SENSORS-2:U5: L3GD20H, L3GD20H:L3GD20H
- added SENSORS-2:U7: MAG3110, MAG3110:MAG3110
- added SENSORS-2:U8: MMA8451Q, MMA8451Q:MMA8451Q
- added SENSORS-2:U9: SI7021, SI7021:SI7021
- added USB:FB1: 600R/1A, SparkFun-Passives:0603
- added USB:J7: ZX62-AB-5PA(31)MICRO-AB-SMT, ZX62-AB-5PA(31):ZX62-AB-5PA(31)
- FD1, FD2, FD3, FD4, FD5: value FIDUCIAL -> FIDUCIAL1X2; device adafruit:FIDUCIAL_1MM -> SparkFun-Aesthetics:FIDUCIAL-1X2
- J1: value CORTEX_DEBUG_SMD -> (none); device SparkFun-Connectors:SAMTECH_FTSH-105-01 -> SparkFun-Connectors:JST-2-SMD
- J2: value DF40FC-20DP-0.4V(51) -> (none); device DF40FC-20DP-0.4V(51):DF40C-20DP-0.4V(51) -> SparkFun-Connectors:JST-2-SMD
- J3: value DF40FC-20DP-0.4V(51) -> QIIC connector; device DF40FC-20DP-0.4V(51):DF40C-20DP-0.4V(51) -> SparkX:1X04_1MM_RA
- J4, J5: value DF40FC-20DP-0.4V(51)SOCKET -> DF40FC-20DP-0.4V(51); device DF40C-20DS-0.4V(51):DF40C-20DP-0.4V(51) -> DF40FC-20DP-0.4V(51):DF40C-20DP-0.4V(51)
- S1: value CHS04SLIDESWITCHA-PKG-VARIANT -> CHS-02_SWITCH; device CHS04SLIDESWITCH:CHS04SLIDESWITCH -> CHS_SWITCH:CHS-02_SWITCH
- S2: value CHS04SLIDESWITCHA-PKG-VARIANT -> CHS-04_SWITCH; device CHS04SLIDESWITCH:CHS04SLIDESWITCH -> CHS_SWITCH:CHS-04_SWITCH
- moved FD3 1471.9 mm to (-499.1, -1313.2), flipped to the top
- moved FD1 1470.1 mm to (-498.9, -1311.4)
- moved FD4 1456.0 mm to (-499.9, -1318.5), flipped to the top
- moved FD2 1421.1 mm to (-499.6, -1316.7)
- moved FD5 1420.8 mm to (-499.4, -1315.0), flipped to the top
- moved J3 1340.9 mm to (-451.1, -1222.2)
- moved J5 1333.0 mm to (-445.0, -1200.2), flipped to the top
- moved J4 1323.0 mm to (-445.0, -1192.5), flipped to the top
- moved S2 1224.0 mm to (-416.6, -1103.1)
- moved J2 1217.5 mm to (-407.2, -1103.9)
- moved S1 953.6 mm to (-293.6, -897.6), turned to 0 degrees
- moved J1 439.4 mm to (-433.8, 88.4), turned to 0 degrees
Connections:
- removed net 25570_LBOOST: L3.2, U21.20
- removed net 25570_LBUCK: L2.1, U21.16
- removed net 25570_OK_HYST: R17.1, R19.2, U21.10
- removed net 25570_OK_PROG: R18.2, R19.1, U21.11
- removed net 25570_VBAT_OV: R16.1, R20.2, U21.7
- removed net 25570_VOUT: C49.1, C51.1, C52.1, C53.1, J2.P$11, L2.2, R40.2, R6.2, U20.10, U20.5, U20.8, U21.14, U22.7, U22.8, U23.10, U23.5, U23.8
- removed net 25570_VOUT_SET: R21.1, R22.2, U21.12
- removed net 25570_VRDIV: R16.2, R17.2, R21.2, U21.8
- removed net 25570_VREF_SAMP: C45.1, U21.4
- removed net 25570_VSTOR: C42.1, C43.1, U21.19, U21.3, U21.6
- removed net ADXL362_CS: J3.P$14, R35.1, U1.P$8, U15.P$14, U22.1
- removed net FT4222_DM: J7.2, U18.P$22
- removed net FT4222_DP: J7.3, U18.P$23
- removed net FT4222_VBUS: C59.1, C60.1, C61.1, C66.1, FB1.1, R24.2, U18.P$26
- removed net FT4222_VOUT3V3: C55.1, C56.1, C57.1, C58.1, R23.1, R5.2, R8.1, S2.1, S2.2, S2.3, S4.2, S4.3, U18.P$1, U18.P$25, U18.P$7
- removed net ICE40_CRESET_B: R43.1, S4.1', U24.8
- removed net ICE40_PIN02: LED4.A, U24.2
- removed net ICE40_PIN03: U24.3
- removed net ICE40_PIN04: U24.4
- removed net ICE40_PIN06: U24.6
- removed net ICE40_PIN07: U24.7
- removed net ICE40_PIN09: U24.9
- removed net ICE40_PIN10: U24.10
- removed net ICE40_PIN11: U24.11
- removed net ICE40_PIN12: U24.12
- removed net ICE40_PIN13: U24.13
- removed net ICE40_PIN14: R36.1, U24.14
- removed net ICE40_PIN15: R37.1, U24.15
- removed net ICE40_PIN16: R38.1, R42.2, U24.16
- removed net ICE40_PIN17: R39.1, U24.17
- removed net ICE40_PIN18: U24.18
- removed net ICE40_PIN19: U24.19
- removed net ICE40_PIN20: U24.20
- removed net ICE40_PIN21: U24.21
- removed net ICE40_PIN23: U24.23
- removed net ICE40_PIN25: U24.25
- removed net ICE40_PIN26: U24.26
- removed net ICE40_PIN27: U24.27
- removed net ICE40_PIN28: U24.28
- removed net ICE40_PIN31: U24.31
- removed net ICE40_PIN32: U24.32
- removed net ICE40_PIN34: U24.34
- removed net ICE40_PIN35: U24.35
- removed net ICE40_PIN36: U24.36
- removed net ICE40_PIN37: U24.37
- removed net ICE40_PIN38: U24.38
- removed net ICE40_PIN39: U24.39
- removed net ICE40_PIN40: U24.40
- removed net ICE40_PIN41: U24.41
- removed net ICE40_PIN42: U24.42
- removed net ICE40_PIN43: U24.43
- removed net ICE40_PIN44: U24.44
- removed net ICE40_PIN45: U24.45
- removed net ICE40_PIN46: U24.46
- removed net ICE40_PIN47: U24.47
- removed net ICE40_PIN48: U24.48
- removed net ICE40_VCCIO: C67.1, C74.1, C75.1, C76.1, C77.1, C78.1, C79.1, C80.1, C81.1, C82.1, R43.2, S4.3', S4.4', U24.1, U24.22, U24.33, U25.4, U25.6
- removed net ICE40_VCC_1V2: C68.1, C69.1, C70.1, C71.1, U24.30, U24.5, U25.1
- removed net ICE40_VCC_PLL: C72.1, C73.1, U24.29
- removed net ICE40_VPP2V5: S4.2', U24.24
- removed net ISL23415_!CS: J3.P$15, R34.1, U15.P$10, U20.4, U23.4
- removed net J4_01: J4.P$1
- removed net J4_02: J4.P$2
- removed net J4_03: J4.P$3
- removed net J4_04: J4.P$4
- removed net J4_05: J4.P$5
- removed net J4_06: J4.P$6
- removed net J4_07: J4.P$7
- removed net J4_08: J4.P$8
- removed net J4_09: J4.P$9
- removed net J4_10: J4.P$10
- removed net J4_11: J4.P$11
- removed net J4_12: J4.P$12
- removed net J4_13: J4.P$13
- removed net J4_14: J4.P$14
- removed net J4_15: J4.P$15
- removed net J4_16: J4.P$16
- removed net J4_17: J4.P$17
- removed net J4_18: J4.P$18
- removed net J4_19: J4.P$19
- removed net J4_20: J4.P$20
- removed net J5_01: J5.P$1
- removed net J5_02: J5.P$2
- removed net J5_03: J5.P$3
- removed net J5_04: J5.P$4
- removed net J5_05: J5.P$5
- removed net J5_06: J5.P$6
- removed net J5_07: J5.P$7
- removed net J5_08: J5.P$8
- removed net J5_09: J5.P$9
- removed net J5_10: J5.P$10
- removed net J5_11: J5.P$11
- removed net J5_12: J5.P$12
- removed net J5_13: J5.P$13
- removed net J5_14: J5.P$14
- removed net J5_15: J5.P$15
- removed net J5_16: J5.P$16
- removed net J5_17: J5.P$17
- removed net J5_18: J5.P$18
- removed net J5_19: J5.P$19
- removed net J5_20: J5.P$20
- removed net KL03_EXTAL0: C31.1, U15.P$5, Y1.P$1
- removed net KL03_I2C0_SCL/KL03_LPUART0_TX: J3.P$10, J6.4, R31.1, S4.1, U10.P$2, U11.3, U12.P$5, U13.P$7, U15.P$17, U16.P$2, U17.10, U2.4, U20.6, U3.P$9, U4.A1, U5.P$2, U7.P$7, U8.P$4, U9.P$6
- removed net KL03_I2C0_SDA/KL03_LPUART0_RX: J3.P$9, J6.3, R32.1, R38.2, U10.P$6, U11.2, U12.P$6, U13.P$8, U15.P$18, U16.P$4, U17.9, U2.3, U23.6, U3.P$11, U4.A2, U5.P$3, U7.P$6, U8.P$6, U9.P$1
- removed net KL03_PTB1: R27.1, U15.P$13
- removed net KL03_RESET_B: J1.10, J3.P$6, R10.1, S3.A, S3.A', U15.P$23
- removed net KL03_SPI_MISO/PAN1326_RTS: J3.P$12, R29.1, R36.2, U1.P$7, U12.P$4, U15.P$8, U22.2, U23.2
- removed net KL03_SPI_MOSI/PAN1326_CTS: J3.P$11, R30.1, R39.2, U1.P$6, U12.P$3, U15.P$11, U20.3, U22.5
- removed net KL03_SPI_SCK: J3.P$13, R28.1, R37.2, U1.P$4, U15.P$12, U20.1, U22.6, U23.1
- removed net KL03_SWD_CLK: J1.4, J3.P$5, R12.1, U15.P$22
- removed net KL03_SWD_DIO: J1.2, J3.P$7, R11.1, U15.P$24
- removed net KL03_VDD: C36.1, C37.1, C54.1, J1.1, R13.2, R14.2, R15.2, R6.1, R7.1, TP25.TP, U14.A2, U15.P$3
- removed net KL03_XTAL0: C25.1, U15.P$6, Y1.P$2
- removed net N$10: C63.1, R9.2, U18.P$21
- removed net N$104: C14.1, U8.P$2
- removed net N$11: C41.2, R4.2
- removed net N$12: FB1.2, J7.1
- removed net N$125: C21.1, U7.P$1
- removed net N$126: C20.1, U7.P$4
- removed net N$13: C65.1, R25.2, U18.P$19, Y2.1
- removed net N$14: C40.1, U11.12
- removed net N$15: C41.1, U11.10
- removed net N$159: C24.1, U5.P$14
- removed net N$16: R25.1, R26.2, U18.P$18
- removed net N$17: C64.1, R26.1, Y2.3
- removed net N$18: R28.2, U18.P$8
- removed net N$19: R29.2, U18.P$9
- removed net N$20: R30.2, U18.P$10
- removed net N$21: R31.2, U18.P$13
- removed net N$22: R24.1, U18.P$30
- removed net N$23: R32.2, U18.P$14
- removed net N$24: R33.2, U18.P$15
- removed net N$25: R34.2, U18.P$16
- removed net N$26: R35.2, U18.P$17
- removed net N$27: R40.1, U22.3
- removed net N$3: LED3.C, R3.2
- removed net N$30: LED4.C, R41.1
- removed net N$32: U25.3
- removed net N$36: R23.2, U18.P$32
- removed net N$6: U17.4, U17.5
- removed net N$7: R8.2, U18.P$2
- removed net N$8: C62.1, R5.1, U18.P$3
- removed net PAN1326B_AUD_CLK: J2.P$12, U12.P$19, U13.P$17
- removed net PAN1326B_AUD_FSYNC: J2.P$14, U12.P$7, U13.P$16
- removed net PAN1326B_AUD_IN: J2.P$13, U12.P$18, U13.P$15
- removed net PAN1326B_AUD_OUT: TP20.TP, U12.P$17
- removed net PAN1326B_RF: TP21.TP, U12.P$13
- removed net PAN1326B_TX_DBG: TP19.TP, U12.P$2
- removed net SCALED_SENSOR_SUPPLY: C10.1, C11.1, C12.1, C13.1, C15.1, C16.1, C17.1, C18.1, C19.1, C22.1, C23.1, C26.1, C27.1, C28.1, C29.1, C3.1, C30.1, C32.1, C33.1, C34.1, C35.1, C38.1, C39.1, C46.1, C47.1, C48.1, C50.1, J2.P$4, J3.P$4, J6.2, S1.3', S2.2', S4.4, U1.P$1, U1.P$14, U10.P$1, U11.13, U11.9, U12.P$10, U12.P$11, U12.P$15, U12.P$22, U13.P$10, U13.P$11, U16.P$1, U16.P$10, U16.P$6, U17.2, U17.6, U2.2, U2.5, U2.6, U2.8, U3.P$13, U3.P$3, U3.P$7, U4.B1, U4.C1, U4.D1, U5.P$1, U5.P$15, U5.P$16, U5.P$5, U7.P$2, U7.P$8, U8.P$1, U8.P$14, U9.P$5
- removed net SI4705_!RST: J2.P$5, LED3.A, R33.1, U13.P$5, U15.P$2
- removed net SI4705_GPO1: J2.P$19, LED1.A, U13.P$19
- removed net SI4705_GPO2: J2.P$18, LED2.A, U13.P$18
- removed net SI4705_LOUT: J2.P$16, U13.P$14
- removed net SI4705_LPI: J2.P$15, U13.P$4
- removed net SI4705_ROUT: J2.P$17, U13.P$13
- removed net SOLAR_VPLUS: D1.+, S1.2
- removed net TPS82740A_CTL/TPS82740A_EN: J3.P$16, U15.P$16, U6.B2, U6.B3
- removed net TPS82740A_LOAD: U6.B1
- removed net TPS82740A_VOUT: U14.B2, U6.C1
- removed net TPS82740B_CTL/TPS82740B_EN: J3.P$17, U15.P$20, U19.B2, U19.B3
- removed net TPS82740B_LOAD: U19.B1
- removed net TPS82740B_VOUT: U14.C2, U19.C1
- removed net TPS82740_DUO_IN: S1.4', U19.C3, U6.C3
- removed net TPS82740_VSEL1: J3.P$18, R13.1, U15.P$7, U19.A3, U6.A3
- removed net TPS82740_VSEL2: J3.P$19, R14.1, U15.P$15, U19.A2, U6.A2
- removed net TPS82740_VSEL3: J3.P$20, R15.1, U15.P$19, U19.A1, U6.A1
- removed net TS5A3154_IN: J2.P$7, U14.D2, U15.P$1
- removed net TS5A3154_OUT: S1.3, U14.A1
- removed net U20_SO: U20.2, U23.3
- removed net VBATT: C1.+, C2.+, C4.+, C5.+, C6.+, C7.+, C8.+, C9.+, J2.P$2, J3.P$2, R10.2, R11.2, R27.2, R7.2, S1.1', S1.4, S2.1'
- removed net VPP: U18.P$29
- removed net WARP_VBOOST_IN: C44.1, L3.1, S1.2', S2.3', U21.2
- removed net WARP_VBOOST_OUT: S1.1, U21.18
- new net ADXL362_FT4222_SPI_CS: FT4222:U18.P$17, J4.P$18, MPU:U1.P$15, SENSORS-1:U1.P$8
- new net BAT: CHARGER:C3.1, CHARGER:TP1.TP, CHARGER:U$1.2, CHARGER:U$1.3, J1.2
- new net BOOST:LBOOST: BOOST:L2.2, BOOST:U21.20
- new net BOOST:LBUCK: BOOST:L3.1, BOOST:U21.16
- new net BOOST:OK_HYST: BOOST:R17.1, BOOST:R19.2, BOOST:U21.10
- new net BOOST:OK_PROG: BOOST:R18.2, BOOST:R19.1, BOOST:U21.11
- new net BOOST:VBAT_OV: BOOST:R16.1, BOOST:R20.2, BOOST:U21.7
- new net BOOST:VOUT_SET: BOOST:R21.1, BOOST:R22.2, BOOST:U21.12
- new net BOOST:VRDIV: BOOST:R16.2, BOOST:R17.2, BOOST:R21.2, BOOST:U21.8
- new net BOOST:VREF_SAMP: BOOST:C45.1, BOOST:U21.4
- new net BOOST:VSTOR: BOOST:C42.1, BOOST:C43.1, BOOST:TP4.TP, BOOST:U21.19, BOOST:U21.3, BOOST:U21.6
- new net BOOST_EN: BOOST:U21.5, S2.1', S2.2'
- new net BOOST_VBAT: BOOST:C1.+, BOOST:C2.+, BOOST:C4.+, BOOST:C5.+, BOOST:C6.+, BOOST:C7.+, BOOST:C8.+, BOOST:C9.+, BOOST:TP3.TP, BOOST:U21.18, S2.2
- new net BOOST_VOUT: BOOST:C49.1, BOOST:L3.2, BOOST:TP2.TP, BOOST:U21.14, S2.3
- new net CHARGER:N$1: CHARGER:R2.2, CHARGER:U$1.16
- new net CHARGER:N$2: CHARGER:R1.2, CHARGER:U$1.12
- new net CHARGER:N$3: CHARGER:R4.1, CHARGER:U$1.7
- new net CHARGER:N$4: CHARGER:R3.2, CHARGER:U$1.1
- new net CHARGER:N$5: CHARGER:R5.1, CHARGER:U$1.9
- new net CHARGER:N$6: CHARGER:D1.C, CHARGER:R4.2
- new net CHARGER:N$7: CHARGER:D2.C, CHARGER:R5.2
- new net CHARGER:N$8: CHARGER:R6.2, CHARGER:U$1.14
- new net CHARGE_VOUT: CHARGER:C2.1, CHARGER:D1.A, CHARGER:D2.A, CHARGER:TP2.TP, CHARGER:U$1.10, CHARGER:U$1.11, S2.4
- new net DF40_SOCKETS:P10A: DF40_SOCKETS:J1.P$10
- new net DF40_SOCKETS:P10B: DF40_SOCKETS:J2.P$10
- new net DF40_SOCKETS:P11A: DF40_SOCKETS:J1.P$11
- new net DF40_SOCKETS:P11B: DF40_SOCKETS:J2.P$11
- new net DF40_SOCKETS:P12A: DF40_SOCKETS:J1.P$12
- new net DF40_SOCKETS:P12B: DF40_SOCKETS:J2.P$12
- new net DF40_SOCKETS:P13A: DF40_SOCKETS:J1.P$13
- new net DF40_SOCKETS:P13B: DF40_SOCKETS:J2.P$13
- new net DF40_SOCKETS:P14A: DF40_SOCKETS:J1.P$14
- new net DF40_SOCKETS:P14B: DF40_SOCKETS:J2.P$14
- new net DF40_SOCKETS:P15A: DF40_SOCKETS:J1.P$15
- new net DF40_SOCKETS:P15B: DF40_SOCKETS:J2.P$15
- new net DF40_SOCKETS:P16A: DF40_SOCKETS:J1.P$16
- new net DF40_SOCKETS:P16B: DF40_SOCKETS:J2.P$16
- new net DF40_SOCKETS:P17A: DF40_SOCKETS:J1.P$17
- new net DF40_SOCKETS:P17B: DF40_SOCKETS:J2.P$17
- new net DF40_SOCKETS:P18A: DF40_SOCKETS:J1.P$18
- new net DF40_SOCKETS:P18B: DF40_SOCKETS:J2.P$18
- new net DF40_SOCKETS:P19A: DF40_SOCKETS:J1.P$19
- new net DF40_SOCKETS:P19B: DF40_SOCKETS:J2.P$19
- new net DF40_SOCKETS:P1A: DF40_SOCKETS:J1.P$1
- new net DF40_SOCKETS:P1B: DF40_SOCKETS:J2.P$1
- new net DF40_SOCKETS:P20A: DF40_SOCKETS:J1.P$20
- new net DF40_SOCKETS:P20B: DF40_SOCKETS:J2.P$20
- new net DF40_SOCKETS:P2A: DF40_SOCKETS:J1.P$2
- new net DF40_SOCKETS:P2B: DF40_SOCKETS:J2.P$2
- new net DF40_SOCKETS:P3A: DF40_SOCKETS:J1.P$3
- new net DF40_SOCKETS:P3B: DF40_SOCKETS:J2.P$3
- new net DF40_SOCKETS:P4A: DF40_SOCKETS:J1.P$4
- new net DF40_SOCKETS:P4B: DF40_SOCKETS:J2.P$4
- new net DF40_SOCKETS:P5A: DF40_SOCKETS:J1.P$5
- new net DF40_SOCKETS:P5B: DF40_SOCKETS:J2.P$5
- new net DF40_SOCKETS:P6A: DF40_SOCKETS:J1.P$6
- new net DF40_SOCKETS:P6B: DF40_SOCKETS:J2.P$6
- new net DF40_SOCKETS:P7A: DF40_SOCKETS:J1.P$7
- new net DF40_SOCKETS:P7B: DF40_SOCKETS:J2.P$7
- new net DF40_SOCKETS:P8A: DF40_SOCKETS:J1.P$8
- new net DF40_SOCKETS:P8B: DF40_SOCKETS:J2.P$8
- new net DF40_SOCKETS:P9A: DF40_SOCKETS:J1.P$9
- new net DF40_SOCKETS:P9B: DF40_SOCKETS:J2.P$9
- new net FPGA:CRESET_B: FPGA:R43.1, FPGA:U$7.F3
- new net FPGA:ICE40_VCC_PLL: FPGA:C5.1, FPGA:C6.1, FPGA:R27.1, FPGA:U$7.B2
- new net FPGA:IOB_0A: FPGA:D1.A, FPGA:U$7.E5
- new net FPGA:IOB_35B_SPI_SS: FPGA:R42.2
- new net FPGA:N$1: FPGA:D1.C, FPGA:R41.1
- new net FPGA:N$2: FPGA:L1.1, FPGA:U$1.A1
- new net FPGA:VCC_1V2: FPGA:L1.2, FPGA:R27.2, FPGA:TP11.TP, FPGA:U$1.C2, FPGA:U$7.C2
- new net FPGA_CS: FPGA:U$7.C1, MPU:U1.P$7
- new net FPGA_VS: FPGA:C10.1, FPGA:C11.1, FPGA:C12.1, FPGA:C13.1, FPGA:C14.1, FPGA:C3.1, FPGA:C4.1, FPGA:C76.1, FPGA:C79.1, FPGA:R43.2, FPGA:U$1.B1, FPGA:U$7.A3, FPGA:U$7.C4, FPGA:U$7.D2, FPGA:U$7.D4, S1.1', S1.2'
- new net FT4222:FT4222_VOUT3V3: FT4222:U18.P$25
- new net FT4222:GPIO2: FT4222:U18.P$15
- new net FT4222:GPIO3: FT4222:U18.P$16
- new net FT4222:N$15: FT4222:C65.1, FT4222:R25.2, FT4222:U18.P$19, FT4222:Y2.1
- new net FT4222:N$2: FT4222:R23.2, FT4222:U18.P$32
- new net FT4222:N$3: FT4222:R8.2, FT4222:U18.P$2
- new net FT4222:N$4: FT4222:C62.1, FT4222:R5.1, FT4222:U18.P$3
- new net FT4222:N$5: FT4222:C63.1, FT4222:R9.2, FT4222:U18.P$21
- new net FT4222:N$6: FT4222:C64.1, FT4222:R25.1, FT4222:U18.P$18, FT4222:Y2.3
- new net FT4222:VPP: FT4222:U18.P$29
- new net I2C0_SCL/UART_TX: FT4222:U18.P$13, J3.4, J4.P$11, MPU:U1.P$17, RF:U12.P$5, RTC:U$5.8
- new net I2C0_SDA/UART_RX: FT4222:U18.P$14, J3.3, J4.P$12, MPU:U1.P$18, RF:U12.P$6, RTC:U$5.1
- new net I2C1_SCL: FPGA:U$7.C3, J4.P$13, SENSORS-1:U10.P$2, SENSORS-1:U11.3, SENSORS-1:U17.10, SENSORS-1:U2.4, SENSORS-1:U20.6, SENSORS-1:U3.P$9
- new net I2C1_SDA: FPGA:U$7.F4, J4.P$14, SENSORS-1:U10.P$6, SENSORS-1:U11.2, SENSORS-1:U17.9, SENSORS-1:U2.3, SENSORS-1:U23.6, SENSORS-1:U3.P$11
- new net I2C2_SCL: FPGA:U$7.A2, J4.P$15, RF:U13.P$7, SENSORS-2:U16.P$2, SENSORS-2:U4.A1, SENSORS-2:U5.P$2, SENSORS-2:U7.P$7, SENSORS-2:U8.P$4, SENSORS-2:U9.P$6
- new net I2C2_SDA: FPGA:U$7.A1, J4.P$16, RF:U13.P$8, SENSORS-2:U16.P$4, SENSORS-2:U4.A2, SENSORS-2:U5.P$3, SENSORS-2:U7.P$6, SENSORS-2:U8.P$6, SENSORS-2:U9.P$1
- new net IOB_12A_G4_CDONE: FPGA:U$7.D3
- new net IOB_13B: FPGA:U$7.E3
- new net IOB_24A: FPGA:U$7.B1
- new net IOB_25B_G3: FPGA:U$7.F2
- new net IOB_2A: FPGA:U$7.D5
- new net IOB_3B_G6: FPGA:U$7.F5
- new net IOB_9B: FPGA:U$7.E4
- new net IOT_46B_G0: FPGA:U$7.B3
- new net IOT_47A: FPGA:U$7.A4
- new net ISL23415_SPI_CS: J4.P$17, MPU:U1.P$20, SENSORS-1:U20.4, SENSORS-1:U23.4
- new net MPU:AT45DB321F_SPI_CS: MPU:U$1.4, MPU:U1.P$16
- new net MPU:EXTAL0: MPU:C31.1, MPU:U1.P$5, MPU:Y1.P$1
- new net MPU:N$4: MPU:R7.1, MPU:U$1.5
- new net MPU:N$5: MPU:C37.2
- new net MPU:N$6: MPU:C36.2
- new net MPU:XTAL0: MPU:C25.1, MPU:U1.P$6, MPU:Y1.P$2
- new net PV_VS: BOOST:C44.1, BOOST:L2.1, BOOST:TP1.TP, BOOST:U21.2, J2.2, J5.P$2
- new net REG:SW: REG:L2.1, REG:U1.2
- new net REG_CTRL: MPU:U1.P$19, REG:R14.2, REG:U1.4
- new net REG_VIN: REG:C2.1, REG:U1.1, REG:U1.12, S2.3', S2.4'
- new net REG_VSEL1: MPU:U1.P$1, REG:R44.2, REG:U1.11
- new net REG_VSEL2: MPU:U1.P$2, REG:R45.2, REG:U1.10
- new net REG_VSEL3: MPU:U1.P$9, REG:R46.2, REG:U1.9
- new net REG_VSEL4: MPU:U1.P$10, REG:R15.2, REG:U1.8
- new net RF:N$1: RF:C32.2
- new net RF:N$2: RF:C33.2
- new net RF:N$3: RF:C35.2
- new net RF:N$4: RF:C34.2
- new net RF:PAN1326_AUD_CLK: RF:U12.P$19, RF:U13.P$17
- new net RF:PAN1326_AUD_FSYNC: RF:U12.P$7, RF:U13.P$16
- new net RF:PAN1326_AUD_IN: RF:U12.P$18, RF:U13.P$15
- new net RF:PAN1326_AUD_OUT: RF:TP20.TP, RF:U12.P$17
- new net RF:PAN1326_RF: RF:TP21.TP, RF:U12.P$13
- new net RF:PAN1326_TX_DBG: RF:TP19.TP, RF:U12.P$2
- new net RF:SI4705_GPO1: RF:U13.P$19
- new net RF:SI4705_GPO2: RF:U13.P$18
- new net RF:SI4705_LPI: RF:TP1.TP, RF:U13.P$4
- new net RGB0: FPGA:U$7.A5
- new net RGB1: FPGA:U$7.B5
- new net RGB2: FPGA:U$7.C5
- new net RTC:N$1: RTC:C1.1, RTC:D2.C, RTC:D3.3, RTC:U$5.3
- new net RTC:N$3: RTC:R6.1, RTC:U$5.7
- new net RTC:VBB: RTC:D2.A, RTC:TP12.TP, RTC:U$6.1, RTC:U$6.3
- new net RTC_!INT!/RESET_B: J4.P$7, J5.P$5, MPU:J1.10, MPU:R10.1, MPU:S3.A, MPU:S3.A', MPU:U1.P$23, RTC:R40.1, RTC:U$5.6
- new net SENSORS-1:N$10: SENSORS-1:C12.2
- new net SENSORS-1:N$11: SENSORS-1:C13.2
- new net SENSORS-1:N$18: SENSORS-1:C28.2
- new net SENSORS-1:N$19: SENSORS-1:C29.2
- new net SENSORS-1:N$20: SENSORS-1:C3.2
- new net SENSORS-1:N$21: SENSORS-1:C30.2
- new net SENSORS-1:N$22: SENSORS-1:C40.2
- new net SENSORS-1:N$23: SENSORS-1:R4.1
- new net SENSORS-1:N$24: SENSORS-1:C52.2
- new net SENSORS-1:N$25: SENSORS-1:C50.2
- new net SENSORS-1:N$27: SENSORS-1:C53.2
- new net SENSORS-1:N$7: SENSORS-1:U17.4, SENSORS-1:U17.5
- new net SENSORS-1:N$8: SENSORS-1:C10.2
- new net SENSORS-1:N$9: SENSORS-1:C11.2
- new net SENSORS-2:N$1: SENSORS-2:C14.1, SENSORS-2:U8.P$2
- new net SENSORS-2:N$11: SENSORS-2:U5.P$5
- new net SENSORS-2:N$12: SENSORS-2:C15.2, SENSORS-2:C48.2
- new net SENSORS-2:N$13: SENSORS-2:C23.2
- new net SENSORS-2:N$14: SENSORS-2:C22.2
- new net SENSORS-2:N$17: SENSORS-2:C20.1, SENSORS-2:C21.1, SENSORS-2:U7.P$1, SENSORS-2:U7.P$4
- new net SENSORS-2:N$18: SENSORS-2:C38.2, SENSORS-2:C39.2
- new net SENSORS-2:N$2: SENSORS-2:C14.2
- new net SENSORS-2:N$27: SENSORS-2:C16.2
- new net SENSORS-2:N$28: SENSORS-2:C17.2
- new net SENSORS-2:N$6: SENSORS-2:C46.2, SENSORS-2:C47.2
- new net SI4705_!RST!: J4.P$19, MPU:U1.P$14, RF:U13.P$5
- new net SPI_MISO/UART_RTS: FPGA:U$7.F1, FT4222:U18.P$9, J4.P$9, MPU:U$1.1, MPU:U1.P$11, RF:U12.P$4, SENSORS-1:U1.P$7, SENSORS-1:U20.2, SENSORS-1:U23.2
- new net SPI_MOSI/UART_CTS: FPGA:U$7.E1, FT4222:U18.P$10, J4.P$10, MPU:U$1.8, MPU:U1.P$8, RF:U12.P$3, SENSORS-1:U1.P$6, SENSORS-1:U20.3, SENSORS-1:U23.3
- new net SPI_SCK: FPGA:U$7.D1, FT4222:U18.P$8, J4.P$8, MPU:U$1.2, MPU:U1.P$12, SENSORS-1:U1.P$4, SENSORS-1:U20.1, SENSORS-1:U23.1
- new net SWD_CLK: J4.P$6, J5.P$4, MPU:J1.4, MPU:R12.1, MPU:U1.P$22
- new net SWD_DIO: J4.P$5, J5.P$3, MPU:J1.2, MPU:R11.1, MPU:U1.P$24
- new net USB:VBUS: USB:FB1.2, USB:J7.1
- new net USB_5V: CHARGER:C1.1, CHARGER:U$1.13, FPGA:C2.1, FPGA:U$1.A2, FT4222:C1.1, FT4222:C2.1, FT4222:U18.P$26, FT4222:U18.P$30, J4.P$2, USB:C61.1, USB:C66.1, USB:FB1.1, USB:TP1.TP
- new net VCC: J3.2
- new net VS_PRI: FT4222:R23.1, FT4222:R5.2, FT4222:R8.1, FT4222:U18.P$1, FT4222:U18.P$7, J4.P$4, MPU:C36.1, MPU:C37.1, MPU:C51.1, MPU:J1.1, MPU:R10.2, MPU:R11.2, MPU:R7.2, MPU:TP25.TP, MPU:U$1.3, MPU:U$1.6, MPU:U1.P$3, REG:C1.1, REG:L2.2, REG:U1.5, RTC:D3.1, RTC:D3.2, RTC:R40.2, RTC:R6.2, S1.1
- new net VS_SEC: J4.P$3, REG:U1.6, RF:C32.1, RF:C33.1, RF:C34.1, RF:C35.1, RF:U12.P$10, RF:U12.P$11, RF:U12.P$15, RF:U12.P$22, RF:U13.P$10, RF:U13.P$11, S1.2, SENSORS-1:C10.1, SENSORS-1:C11.1, SENSORS-1:C12.1, SENSORS-1:C13.1, SENSORS-1:C26.1, SENSORS-1:C27.1, SENSORS-1:C28.1, SENSORS-1:C29.1, SENSORS-1:C3.1, SENSORS-1:C30.1, SENSORS-1:C40.1, SENSORS-1:C50.1, SENSORS-1:C52.1, SENSORS-1:C53.1, SENSORS-1:U1.P$1, SENSORS-1:U1.P$14, SENSORS-1:U10.P$1, SENSORS-1:U11.12, SENSORS-1:U11.13, SENSORS-1:U11.9, SENSORS-1:U17.2, SENSORS-1:U17.6, SENSORS-1:U2.2, SENSORS-1:U2.5, SENSORS-1:U2.6, SENSORS-1:U2.8, SENSORS-1:U20.10, SENSORS-1:U20.5, SENSORS-1:U20.8, SENSORS-1:U23.10, SENSORS-1:U23.5, SENSORS-1:U23.8, SENSORS-1:U3.P$13, SENSORS-1:U3.P$3, SENSORS-1:U3.P$7, SENSORS-2:C15.1, SENSORS-2:C16.1, SENSORS-2:C17.1, SENSORS-2:C18.1, SENSORS-2:C19.1, SENSORS-2:C22.1, SENSORS-2:C23.1, SENSORS-2:C24.1, SENSORS-2:C38.1, SENSORS-2:C39.1, SENSORS-2:C46.1, SENSORS-2:C47.1, SENSORS-2:C48.1, SENSORS-2:U16.P$1, SENSORS-2:U16.P$10, SENSORS-2:U16.P$6, SENSORS-2:U4.B1, SENSORS-2:U4.C1, SENSORS-2:U4.D1, SENSORS-2:U5.P$1, SENSORS-2:U5.P$14, SENSORS-2:U5.P$16, SENSORS-2:U7.P$2, SENSORS-2:U7.P$8, SENSORS-2:U8.P$1, SENSORS-2:U8.P$14, SENSORS-2:U9.P$5
- net GND: now also BOOST:C1.-, BOOST:C2.-, BOOST:C4.-, BOOST:C42.2, BOOST:C43.2, BOOST:C44.2, BOOST:C45.2, BOOST:C49.2, BOOST:C5.-, BOOST:C6.-, BOOST:C7.-, BOOST:C8.-, BOOST:C9.-, BOOST:R18.1, BOOST:R20.1, BOOST:R22.1, BOOST:U21.1, BOOST:U21.15, BOOST:U21.17, BOOST:U21.21, BOOST:U21.9, CHARGER:C1.2, CHARGER:C2.2, CHARGER:C3.2, CHARGER:R1.1, CHARGER:R2.1, CHARGER:R3.1, CHARGER:R6.1, CHARGER:U$1.15, CHARGER:U$1.4, CHARGER:U$1.6, CHARGER:U$1.8, CHARGER:U$1.EP, FPGA:C10.2, FPGA:C11.2, FPGA:C12.2, FPGA:C13.2, FPGA:C14.2, FPGA:C2.2, FPGA:C3.2, FPGA:C4.2, FPGA:C5.2, FPGA:C6.2, FPGA:C76.2, FPGA:C79.2, FPGA:R41.2, FPGA:R42.1, FPGA:U$1.B2, FPGA:U$1.C1, FPGA:U$7.B4, FPGA:U$7.E2, FT4222:C1.2, FT4222:C2.2, FT4222:C62.2, FT4222:C63.2, FT4222:C64.2, FT4222:C65.2, FT4222:R9.1, FT4222:U18.P$20, FT4222:U18.P$24, FT4222:U18.P$27, FT4222:U18.P$28, FT4222:U18.P$4, FT4222:U18.P$5, FT4222:U18.P$6, J1.1, J2.1, J3.1, J4.P$1, J5.P$1, MPU:C25.2, MPU:C31.2, MPU:C51.2, MPU:J1.3, MPU:J1.5, MPU:R12.2, MPU:S3.B, MPU:S3.B', MPU:U$1.7, MPU:U$1.9, MPU:U1.P$4, MPU:U1.P$PAD, REG:C1.2, REG:C2.2, REG:R14.1, REG:R15.1, REG:R44.1, REG:R45.1, REG:R46.1, REG:U1.3, RF:U12.P$1, RF:U12.P$12, RF:U12.P$14, RF:U12.P$20, RF:U13.P$12, RF:U13.P$21, RF:U13.P$3, RF:U13.P$6, RTC:C1.2, RTC:U$5.4, RTC:U$5.5, RTC:U$6.2, S2.1, SENSORS-1:C26.2, SENSORS-1:C27.2, SENSORS-1:C41.1, SENSORS-1:C41.2, SENSORS-1:R4.2, SENSORS-1:U1.P$12, SENSORS-1:U1.P$13, SENSORS-1:U1.P$16, SENSORS-1:U10.P$3, SENSORS-1:U11.10, SENSORS-1:U11.5, SENSORS-1:U11.6, SENSORS-1:U17.1, SENSORS-1:U17.7, SENSORS-1:U17.EP, SENSORS-1:U2.1, SENSORS-1:U2.7, SENSORS-1:U20.9, SENSORS-1:U23.9, SENSORS-1:U3.P$12, SENSORS-1:U3.P$17, SENSORS-1:U3.P$20, SENSORS-1:U3.P$4, SENSORS-1:U3.P$6, SENSORS-2:C18.2, SENSORS-2:C19.2, SENSORS-2:C20.2, SENSORS-2:C21.2, SENSORS-2:C24.2, SENSORS-2:U16.P$3, SENSORS-2:U16.P$5, SENSORS-2:U16.P$8, SENSORS-2:U16.P$9, SENSORS-2:U4.B2, SENSORS-2:U5.P$10, SENSORS-2:U5.P$11, SENSORS-2:U5.P$12, SENSORS-2:U5.P$13, SENSORS-2:U5.P$15, SENSORS-2:U5.P$4, SENSORS-2:U5.P$9, SENSORS-2:U7.P$10, SENSORS-2:U7.P$5, SENSORS-2:U8.P$10, SENSORS-2:U8.P$12, SENSORS-2:U8.P$5, SENSORS-2:U8.P$7, SENSORS-2:U9.P$2, USB:C61.2, USB:C66.2, USB:J7.4, USB:J7.5; no longer C1.-, C10.2, C11.2, C12.2, C13.2, C14.2, C15.2, C16.2, C17.2, C18.2, C19.2, C2.-, C20.2, C21.2, C22.2, C23.2, C24.2, C25.2, C26.2, C27.2, C28.2, C29.2, C3.2, C30.2, C31.2, C32.2, C33.2, C34.2, C35.2, C36.2, C37.2, C38.2, C39.2, C4.-, C40.2, C42.2, C43.2, C44.2, C45.2, C46.2, C47.2, C48.2, C49.2, C5.-, C50.2, C51.2, C52.2, C53.2, C54.2, C55.2, C56.2, C57.2, C58.2, C59.2, C6.-, C60.2, C61.2, C62.2, C63.2, C64.2, C65.2, C66.2, C67.2, C68.2, C69.2, C7.-, C70.2, C71.2, C72.2, C73.2, C74.2, C75.2, C76.2, C77.2, C78.2, C79.2, C8.-, C80.2, C81.2, C82.2, C9.-, D1.-, J1.3, J1.5, J2.P$1, J3.P$1, J6.1, J7.4, J7.5, R1.1, R12.2, R18.1, R2.1, R20.1, R22.1, R3.1, R4.1, R41.2, R42.1, R9.1, S3.B, S3.B', U1.P$12, U1.P$13, U1.P$16, U10.P$3, U11.5, U11.6, U12.P$1, U12.P$12, U12.P$14, U12.P$20, U13.P$12, U13.P$21, U13.P$3, U13.P$6, U14.B1, U14.C1, U14.D1, U15.P$4, U15.P$PAD, U16.P$3, U16.P$5, U16.P$8, U16.P$9, U17.1, U17.7, U17.EP, U18.P$20, U18.P$24, U18.P$27, U18.P$28, U18.P$4, U18.P$5, U18.P$6, U19.C2, U2.1, U2.7, U20.9, U21.1, U21.15, U21.17, U21.21, U21.5, U21.9, U22.4, U23.9, U24.P$1, U25.7, U3.P$12, U3.P$17, U3.P$20, U3.P$4, U3.P$6, U4.B2, U5.P$10, U5.P$11, U5.P$12, U5.P$13, U5.P$4, U5.P$9, U6.C2, U7.P$10, U7.P$5, U8.P$10, U8.P$12, U8.P$5, U8.P$7, U9.P$2
- net KL03_CLKOUT32K: now also MPU:U1.P$21, RF:U12.P$8, RF:U13.P$9; no longer J2.P$6, U12.P$8, U13.P$9, U15.P$21
- net N$1: now also FT4222:U18.P$23, USB:J7.3; no longer LED1.C, R1.2
- net N$2: now also FT4222:U18.P$22, USB:J7.2; no longer LED2.C, R2.2
- net PAN1326_!SHUTD: now also J4.P$20, MPU:U1.P$13, RF:U12.P$16; no longer J2.P$8, U12.P$16, U15.P$9
- net SI4705_FMI: now also J5.P$6, RF:TP2.TP, RF:U13.P$2; no longer J2.P$20, U13.P$2
Routing:
- net GND: track 413.7 -> 0.00 mm, vias 72 -> 5
- net KL03_I2C0_SCL/KL03_LPUART0_TX: track 236.6 -> 0.00 mm, vias 13 -> 0
- net SCALED_SENSOR_SUPPLY: track 226.2 -> 0.00 mm, vias 23 -> 1
- net KL03_I2C0_SDA/KL03_LPUART0_RX: track 224.3 -> 0.00 mm, vias 11 -> 0
- net KL03_SPI_SCK: track 148.1 -> 0.00 mm, vias 6 -> 0
- net KL03_VDD: track 144.9 -> 0.00 mm, vias 6 -> 0
- net KL03_SPI_MISO/PAN1326_RTS: track 139.9 -> 0.00 mm, vias 7 -> 0
- net KL03_SPI_MOSI/PAN1326_CTS: track 119.5 -> 0.00 mm, vias 9 -> 0
- net 25570_VOUT: track 102.2 -> 0.00 mm, vias 6 -> 0
- net FT4222_VOUT3V3: track 96.0 -> 0.00 mm, vias 5 -> 0
- net SOLAR_VPLUS: track 88.4 -> 0.00 mm, vias 2 -> 0
- net WARP_VBOOST_OUT: track 82.8 -> 0.00 mm, vias 2 -> 0
- net SI4705_!RST: track 81.7 -> 0.00 mm, vias 3 -> 0
- net ADXL362_CS: track 72.9 -> 0.00 mm, vias 4 -> 0
- net ISL23415_!CS: track 69.0 -> 0.00 mm, vias 4 -> 0
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- added copper zone on layer 14, net BOOST_VBAT
- added copper zone on layer 1, net BOOST_VIN
- added copper zone on layer 14, net BOOST_VIN
- added copper zone on layer 15, net BOOST_VIN
- added copper zone on layer 16, net BOOST_VIN
- added copper zone on layer 2, net BOOST_VIN
- added copper zone on layer 3, net BOOST_VIN
- added copper zone on layer 4, net BOOST_VIN
- added copper zone on layer 5, net BOOST_VIN
- added copper zone on layer 6, net BOOST_VIN
- added copper zone on layer 7, net BOOST_VIN
- removed copper zone on layer 1, net N$5
- removed copper zone on layer 14, net N$5
- removed copper zone on layer 15, net N$5
- removed copper zone on layer 16, net N$5
- removed copper zone on layer 2, net N$5
- removed copper zone on layer 3, net N$5
- removed copper zone on layer 4, net N$5
- removed copper zone on layer 5, net N$5
- removed copper zone on layer 6, net N$5
- removed copper zone on layer 7, net N$5
- removed copper zone on layer 14, net VBATT
