File: revB/cad/eagle/warp-revB.sch (EAGLE design)
At the start: 180 parts, among them J1 CORTEX_DEBUG_SMD, J2 DF40FC-20DP-0.4V(51), J3 DF40FC-20DP-0.4V(51), J4 DF40FC-20DP-0.4V(51)SOCKET, J5 DF40FC-20DP-0.4V(51)SOCKET, J6 QIIC connector, J7 ZX62-AB-5PA(31)MICRO-AB-SMT, U1 ADXL362, U10 TCS34725FN, U11 GRIDEYE, U12 PAN1326C, U13 SI4705, U14 TS5A3154, U15 MKL03Z32CAF4RQFN24, U16 LPS25H, U17 CCS811, U18 FT4222H, U19 TPS82740B, U2 BME680LGA, U20 ISL23415UTQFN, U21 BQ25570PVQFN, U22 SERIAL-NOR-FLASHWSON-6X5, U23 ISL23415UTQFN, U24 ICE40UP5K-SG48QFN48, U25 TLV757P, U3 BMX055, U4 HDC1000, U5 L3GD20H, U6 TPS82740A, U7 MAG3110, U8 MMA8451Q, U9 SI7021, Y1 CM519-SMD, Y2 CS325

Commit message: solved power issues and added RV8803 support
Parts:
- removed C1, C2, C4, C5, C6, C7, C8, C9: XH414HGIV01E, XH414HGIV01E:XH414HGIV01E
- removed C10, C12, C14, C16, C18, C20, C21, C23, C26, C28, C3, C32, C34, C37, C38, C46, C48, C51, C52, C53, C54, C56, C58, C60, C66, C70, C73, C75, C78, C81: 0.1uF, SparkFun-Passives:CAP0402-CAP
- removed C11, C13, C17, C22, C27, C29, C39, C47, C67, C68, C69, C74, C77, C80: 1uF, SparkFun-Passives:CAP0402-CAP
- removed C15, C30, C33, C72: 10uF, SparkFun-Passives:CAP0402-CAP
- removed C19, C42, C44, C50: 4.7uF, SparkFun-Passives:CAP0402-CAP
- removed C24: 10nF (25V), SparkFun-Passives:CAP0402-CAP
- removed C25, C31: 33pF, SparkFun-Passives:CAP0402-CAP
- removed C35: 22nF, SparkFun-Passives:CAP0402-CAP
- removed C36, C55, C57, C59, C61: 4.7uF (pol), SparkFun-Passives:CAP0402-CAP
- removed C40: 2.2uF, SparkFun-Passives:CAP0402-CAP
- removed C41: 1.0uF, SparkFun-Passives:CAP0402-CAP
- removed C43: 0.01uF, SparkFun-Passives:CAP0402-CAP
- removed C45, C71, C76, C79, C82: 10nF, SparkFun-Passives:CAP0402-CAP
- removed C49: 22uF, SparkFun-Passives:CAP0603-CAP
- removed C62: 0.47uF, SparkFun-Passives:CAP0402-CAP
- removed C63: 100pF, SparkFun-Passives:CAP0402-CAP
- removed C64, C65: 27pF, SparkFun-Passives:CAP0402-CAP
- removed D1: KXOB22-04X3F, KX0B22-04X3F:KXOB22-04X3F
- removed FB1: 600R/1A, SparkFun-Passives:INDUCTOR0603
- removed J6: QIIC connector, SparkX:I2C_STANDARDJS-1MM
- removed J7: ZX62-AB-5PA(31)MICRO-AB-SMT, ZX62-AB-5PA(31):ZX62-AB-5PA(31)MICRO-AB-SMT
- removed L2: 10uH, PowerMagnetics (rev17f):WE-TPC_2813_744029100
- removed L3: 22uH, PowerMagnetics (rev17f):WE-TPC_3816_744031220
- removed LED1, LED2, LED3, LED4: (no value), led:LEDSML0603
- removed R1, R2, R3, R41: 4.7k, SparkFun-Passives:RESISTOR0402-RES
- removed R10: 4.7K, SparkFun-Passives:RESISTOR0402-RES
- removed R11: 10K, SparkFun-Passives:RESISTOR0402-RES
- removed R12, R40, R43: 10k, SparkFun-Passives:RESISTOR0402-RES
- removed R13, R14, R15, R23, R8: 10k, SparkFun-Resistors:RESISTOR0402
- removed R16: 7.32M, SparkFun-Passives:RESISTOR0402-RES
- removed R17: 1.91M, SparkFun-Passives:RESISTOR0402-RES
- removed R18, R20: 5.62M, SparkFun-Passives:RESISTOR0402-RES
- removed R19: 5.49M, SparkFun-Passives:RESISTOR0402-RES
- removed R21: 4.22M, SparkFun-Passives:RESISTOR0402-RES
- removed R22: 8.66M, SparkFun-Passives:RESISTOR0402-RES
- removed R24, R26, R28, R29, R30, R31, R32, R33, R34, R35, R36, R37, R38, R39: 0, SparkFun-Resistors:RESISTOR0402
- removed R25: 1M, SparkFun-Resistors:RESISTOR0402
- removed R27, R7: 0, SparkFun-Passives:RESISTOR0402-RES
- removed R4: 20, SparkFun-Resistors:RESISTOR0402
- removed R42, R6: DNP, SparkFun-Passives:RESISTOR0402-RES
- removed R5: 47k, SparkFun-Resistors:RESISTOR0402
- removed R9: 12k (1%), SparkFun-Resistors:RESISTOR0402
- removed S3: EVPAYG0BAEVPAYG0BA, EVPAYG0BA:EVPAYG0BAEVPAYG0BA
- removed S4: CHS04SLIDESWITCHA-PKG-VARIANT, CHS04SLIDESWITCH:CHS04SLIDESWITCHA-PKG-VARIANT
- removed TP19, TP20, TP21: TPTP06R, testpad:TPTP06R
- removed TP25: TPSTP06R, testpad:TPSTP06R
- removed U1: ADXL362, ADXL362:ADXL362
- removed U10: TCS34725FN, TCS3772:TCS3772
- removed U11: GRIDEYE, Grideye:GRIDEYE
- removed U12: PAN1326C, PAN1326B:PAN1326B
- removed U13: SI4705, SI4705:SI4705
- removed U14: TS5A3154, TS5A3154:TS5A3154
- removed U15: MKL03Z32CAF4RQFN24, MKL03Z32CAF4R:MKL03Z32CAF4RQFN24
- removed U16: LPS25H, LPS25H:LPS25H
- removed U17: CCS811, SparkFun-Sensors:CCS811PRODUCTION
- removed U18: FT4222H, FT4222H:FT4222H
- removed U19: TPS82740B, TPS82740:TPS82740
- removed U2: BME680LGA, BME680:BME680LGA
- removed U20, U23: ISL23415UTQFN, ISL23415:ISL23415UTQFN
- removed U21: BQ25570PVQFN, BQ25570:BQ25570PVQFN
- removed U22: SERIAL-NOR-FLASHWSON-6X5, WSON-6x5:SERIAL-NOR-FLASHWSON-6X5
- removed U24: ICE40UP5K-SG48QFN48, Lattice-QFN48:ICE40UP5K-SG48QFN48
- removed U25: TLV757P, TLV757P:TLV757P
- removed U3: BMX055, BMX055:BMX055
- removed U4: HDC1000, HDC1000:HDC1000
- removed U5: L3GD20H, L3GD20H:L3GD20H
- removed U6: TPS82740A, TPS82740:TPS82740
- removed U7: MAG3110, MAG3110:MAG3110
- removed U8: MMA8451Q, MMA8451Q:MMA8451Q
- removed U9: SI7021, SI7021:SI7021
- removed Y1: CM519-SMD, CM519:CM519-SMD
- removed Y2: CS325, CS325:CS325
- FD1, FD2, FD3, FD4, FD5: value FIDUCIAL -> FIDUCIAL1X2; device adafruit:FIDUCIAL -> SparkFun-Aesthetics:FIDUCIAL1X2
- J1: value CORTEX_DEBUG_SMD -> (none); device SparkFun-Connectors:CORTEX_DEBUG_SMD -> SparkFun-Connectors:JST_2MM_MALE
- J2: value DF40FC-20DP-0.4V(51) -> (none); device DF40FC-20DP-0.4V(51):DF40FC-20DP-0.4V(51) -> SparkFun-Connectors:JST_2MM_MALE
- J3: value DF40FC-20DP-0.4V(51) -> QIIC connector; device DF40FC-20DP-0.4V(51):DF40FC-20DP-0.4V(51) -> SparkX:I2C_STANDARDJS-1MM
- J4, J5: value DF40FC-20DP-0.4V(51)SOCKET -> DF40FC-20DP-0.4V(51); device DF40C-20DS-0.4V(51):DF40FC-20DP-0.4V(51)SOCKET -> DF40FC-20DP-0.4V(51):DF40FC-20DP-0.4V(51)
- S1: value CHS04SLIDESWITCHA-PKG-VARIANT -> CHS-02_SWITCH; device CHS04SLIDESWITCH:CHS04SLIDESWITCHA-PKG-VARIANT -> CHS_SWITCH:CHS-02_SWITCH
- S2: value CHS04SLIDESWITCHA-PKG-VARIANT -> CHS-04_SWITCH; device CHS04SLIDESWITCH:CHS04SLIDESWITCHA-PKG-VARIANT -> CHS_SWITCH:CHS-04_SWITCH
Connections:
- net J4_02 renamed USB_5V
- net J4_08 renamed SPI_SCK
- net J4_09 renamed SPI_MISO/UART_RTS
- net J4_10 renamed SPI_MOSI/UART_CTS
- net J4_13 renamed I2C1_SCL
- net J4_14 renamed I2C1_SDA
- net J4_15 renamed I2C2_SCL
- net J4_16 renamed I2C2_SDA
- net J4_17 renamed ISL23415_SPI_CS
- net J4_18 renamed ADXL362_FT4222_SPI_CS
- net J4_19 renamed SI4705_!RST!
- removed net 25570_LBOOST: L3.2, U21.LBOOST
- removed net 25570_LBUCK: L2.1, U21.LBUCK
- removed net 25570_OK_HYST: R17.1, R19.2, U21.OK_HYST
- removed net 25570_OK_PROG: R18.2, R19.1, U21.OK_PROG
- removed net 25570_VBAT_OV: R16.1, R20.2, U21.VBAT_OV
- removed net 25570_VOUT: C49.1, C51.1, C52.1, C53.1, J2.P$11, L2.2, R40.2, R6.2, U20.RL, U20.VCC, U20.VLOGIC, U21.VOUT, U22.!RESET, U22.VCC, U23.RL, U23.VCC, U23.VLOGIC
- removed net 25570_VOUT_SET: R21.1, R22.2, U21.VOUT_SET
- removed net 25570_VRDIV: R16.2, R17.2, R21.2, U21.VRDIV
- removed net 25570_VREF_SAMP: C45.1, U21.VREF_SAMP
- removed net 25570_VSTOR: C42.1, C43.1, U21.VOC_SAMP, U21.VOUT_EN, U21.VSTOR
- removed net ADXL362_CS: J3.P$14, R35.1, U1.!CS, U15.PTB2/IRQ_7, U22.!CE
- removed net FT4222_DM: J7.DM, U18.DM
- removed net FT4222_DP: J7.DP, U18.DP
- removed net FT4222_VBUS: C59.1, C60.1, C61.1, C66.1, FB1.1, R24.2, U18.VCCIN
- removed net FT4222_VOUT3V3: C55.1, C56.1, C57.1, C58.1, R23.1, R5.2, R8.1, S2.1, S2.2, S2.3, S4.2, S4.3, U18.DEBUGGER, U18.VCCIO, U18.VOUT_3V3
- removed net ICE40_CRESET_B: R43.1, S4.1', U24.CRESET_B
- removed net ICE40_PIN02: LED4.A, U24.IOB_6A
- removed net ICE40_PIN03: U24.IOB_9B
- removed net ICE40_PIN04: U24.IOB_8A
- removed net ICE40_PIN06: U24.IOB_13B
- removed net ICE40_PIN07: U24.CDONE
- removed net ICE40_PIN09: U24.IOB_16A
- removed net ICE40_PIN10: U24.IOB_18A
- removed net ICE40_PIN11: U24.IOB_20A
- removed net ICE40_PIN12: U24.IOB_22A
- removed net ICE40_PIN13: U24.IOB_24A
- removed net ICE40_PIN14: R36.1, U24.IOB_32A_SPI_SO
- removed net ICE40_PIN15: R37.1, U24.IOB_34A_SPI_SCK
- removed net ICE40_PIN16: R38.1, R42.2, U24.IOB_35B_SPI_SS
- removed net ICE40_PIN17: R39.1, U24.IOB_33B_SPI_SI
- removed net ICE40_PIN18: U24.IOB_31B
- removed net ICE40_PIN19: U24.IOB_29B
- removed net ICE40_PIN20: U24.IOB_25B_G3
- removed net ICE40_PIN21: U24.IOB_23B
- removed net ICE40_PIN23: U24.IOT_37A
- removed net ICE40_PIN25: U24.IOT_36B
- removed net ICE40_PIN26: U24.IOT_39A
- removed net ICE40_PIN27: U24.IOT_38B
- removed net ICE40_PIN28: U24.IOT_41A
- removed net ICE40_PIN31: U24.IOT_42B
- removed net ICE40_PIN32: U24.IOT_43A
- removed net ICE40_PIN34: U24.IOT_44B
- removed net ICE40_PIN35: U24.IOT_46B_G0
- removed net ICE40_PIN36: U24.IOT_48B
- removed net ICE40_PIN37: U24.IOT_45A_G1
- removed net ICE40_PIN38: U24.IOT_50B
- removed net ICE40_PIN39: U24.RGB0
- removed net ICE40_PIN40: U24.RGB1
- removed net ICE40_PIN41: U24.RGB2
- removed net ICE40_PIN42: U24.IOT_51A
- removed net ICE40_PIN43: U24.IOT_49A
- removed net ICE40_PIN44: U24.IOB_3B_G6
- removed net ICE40_PIN45: U24.IOB_5B
- removed net ICE40_PIN46: U24.IOB_0A
- removed net ICE40_PIN47: U24.IOB_2A
- removed net ICE40_PIN48: U24.IOB_4A
- removed net ICE40_VCCIO: C67.1, C74.1, C75.1, C76.1, C77.1, C78.1, C79.1, C80.1, C81.1, C82.1, R43.2, S4.3', S4.4', U24.SPI_VCCIO1, U24.VCCIO_0, U24.VCCIO_2, U25.EN, U25.IN
- removed net ICE40_VCC_1V2: C68.1, C69.1, C70.1, C71.1, U24.VCC_PIN30, U24.VCC_PIN5, U25.OUT
- removed net ICE40_VCC_PLL: C72.1, C73.1, U24.VCCPLL
- removed net ICE40_VPP2V5: S4.2', U24.VPP_2V5
- removed net ISL23415_!CS: J3.P$15, R34.1, U15.PTB11, U20.CS, U23.CS
- removed net J4_01: J4.P$1
- removed net J4_03: J4.P$3
- removed net J4_04: J4.P$4
- removed net J4_05: J4.P$5
- removed net J4_06: J4.P$6
- removed net J4_07: J4.P$7
- removed net J4_11: J4.P$11
- removed net J4_12: J4.P$12
- removed net J4_20: J4.P$20
- removed net J5_01: J5.P$1
- removed net J5_02: J5.P$2
- removed net J5_03: J5.P$3
- removed net J5_04: J5.P$4
- removed net J5_05: J5.P$5
- removed net J5_06: J5.P$6
- removed net J5_07: J5.P$7
- removed net J5_08: J5.P$8
- removed net J5_09: J5.P$9
- removed net J5_10: J5.P$10
- removed net J5_11: J5.P$11
- removed net J5_12: J5.P$12
- removed net J5_13: J5.P$13
- removed net J5_14: J5.P$14
- removed net J5_15: J5.P$15
- removed net J5_16: J5.P$16
- removed net J5_17: J5.P$17
- removed net J5_18: J5.P$18
- removed net J5_19: J5.P$19
- removed net J5_20: J5.P$20
- removed net KL03_CLKOUT32K: J2.P$6, U12.SLOW_CLK_IN, U13.RCLK, U15.PTB13/CLKOUT32K
- removed net KL03_EXTAL0: C31.1, U15.PTA3/EXTAL0, Y1.1
- removed net KL03_I2C0_SCL/KL03_LPUART0_TX: J3.P$10, J6.SCL, R31.1, S4.1, U10.SCL, U11.SCL, U12.HCI_RX, U13.SCLK, U15.PTB3/IRQ_10, U16.I2C_SCL/SPI_SPC, U17.SCL, U2.SCK, U20.RW, U3.SCX, U4.SCL, U5.I2C_SCL/SPI_SPC, U7.SCL, U8.SCL, U9.SCL
- removed net KL03_I2C0_SDA/KL03_LPUART0_RX: J3.P$9, J6.SDA, R32.1, R38.2, U10.SDA, U11.SDA, U12.HCI_TX, U13.SDIO, U15.PTB4/IRQ_11, U16.I2C_SDA/SPI4_SDI/SPI3_SDIO, U17.SDA, U2.SDI, U23.RW, U3.SDX, U4.SDA, U5.I2C_SDA/SPI_SDI/SPI3_SDO, U7.SDA, U8.SDA, U9.SDA
- removed net KL03_PTB1: R27.1, U15.PTB1/IRQ_6/ADC0_SE8/CMP0_IN3
- removed net KL03_RESET_B: J1.!RESET, J3.P$6, R10.1, S3.A, S3.A', U15.PTA1/IRQ1/LPTMR0_ALT1
- removed net KL03_SPI_MISO/PAN1326_RTS: J3.P$12, R29.1, R36.2, U1.MISO, U12.HCI_RTS, U15.PTA6, U22.SO, U23.SDO
- removed net KL03_SPI_MOSI/PAN1326_CTS: J3.P$11, R30.1, R39.2, U1.MOSI, U12.HCI_CTS, U15.PTA7/IRQ_4, U20.SDI, U22.SI
- removed net KL03_SPI_SCK: J3.P$13, R28.1, R37.2, U1.SCLK, U15.PTB0/IRQ_5/LLWU_P4, U20.SCK, U22.SCK, U23.SCK
- removed net KL03_SWD_CLK: J1.SWDCLK/TCK, J3.P$5, R12.1, U15.PTA0/IRQ_0/LLWU_P7
- removed net KL03_SWD_DIO: J1.SWDIO/TMS, J3.P$7, R11.1, U15.PTA2
- removed net KL03_VDD: C36.1, C37.1, C54.1, J1.VCC, R13.2, R14.2, R15.2, R6.1, R7.1, TP25.PP, U14.V+, U15.VDD
- removed net KL03_XTAL0: C25.1, U15.PTA4/XTAL0, Y1.2
- removed net N$1: LED1.C, R1.2
- removed net N$10: C63.1, R9.2, U18.RREF
- removed net N$104: C14.1, U8.BYP
- removed net N$11: C41.2, R4.2
- removed net N$12: FB1.2, J7.VBUS
- removed net N$125: C21.1, U7.CAP_A
- removed net N$126: C20.1, U7.CAP_R
- removed net N$13: C65.1, R25.2, U18.XSCO, Y2.P$1
- removed net N$14: C40.1, U11.DVDD
- removed net N$15: C41.1, U11.AVDD
- removed net N$159: C24.1, U5.CAP
- removed net N$16: R25.1, R26.2, U18.XSCI
- removed net N$17: C64.1, R26.1, Y2.P$2
- removed net N$18: R28.2, U18.SCK
- removed net N$19: R29.2, U18.MISO
- removed net N$2: LED2.C, R2.2
- removed net N$20: R30.2, U18.MOSI
- removed net N$21: R31.2, U18.GPIO0/SS1O/SCL
- removed net N$22: R24.1, U18.VBUS_DET
- removed net N$23: R32.2, U18.GPIO1/SS2O/SDA
- removed net N$24: R33.2, U18.GPIO2/SS3O/SUSP_OUT
- removed net N$25: R34.2, U18.GPIO3/WAKEUP/INTR
- removed net N$26: R35.2, U18.SS0O
- removed net N$27: R40.1, U22.!WP
- removed net N$3: LED3.C, R3.2
- removed net N$30: LED4.C, R41.1
- removed net N$32: U25.GND
- removed net N$36: R23.2, U18.SS
- removed net N$6: U17.PWM, U17.SENSE
- removed net N$7: R8.2, U18.!STEST_RSTN
- removed net N$8: C62.1, R5.1, U18.!RESETN
- removed net PAN1326B_AUD_CLK: J2.P$12, U12.AUD_CLK, U13.GPO3/DCLK
- removed net PAN1326B_AUD_FSYNC: J2.P$14, U12.AUD_FSYNC, U13.DFS
- removed net PAN1326B_AUD_IN: J2.P$13, U12.AUD_IN, U13.DOUT
- removed net PAN1326B_AUD_OUT: TP20.TP, U12.AUD_OUT
- removed net PAN1326B_RF: TP21.TP, U12.RF
- removed net PAN1326B_TX_DBG: TP19.TP, U12.TX_DBG
- removed net SCALED_SENSOR_SUPPLY: C10.1, C11.1, C12.1, C13.1, C15.1, C16.1, C17.1, C18.1, C19.1, C22.1, C23.1, C26.1, C27.1, C28.1, C29.1, C3.1, C30.1, C32.1, C33.1, C34.1, C35.1, C38.1, C39.1, C46.1, C47.1, C48.1, C50.1, J2.P$4, J3.P$4, J6.VCC, S1.3', S2.2', S4.4, U1.VDDIO, U1.VS, U10.VDD, U11.VDD, U11.VPP, U12.CL1.5_LDO_IN, U12.MLDO_IN, U12.MLDO_OUT, U12.VDD_IO, U13.VA, U13.VD, U16.I2C_VS_SPI_MODE_SELECT/SPI_EN, U16.VDD, U16.VDD_IO, U17.!RESET!, U17.VDD, U2.CSB, U2.SDO, U2.VDD, U2.VDDIO, U3.PS, U3.VDD, U3.VDDIO, U4.ADR0, U4.ADR1, U4.VDD, U5.I2C_VS_SPI_MODE_SELECT, U5.RESERVED@15, U5.VDD, U5.VDD_IO, U7.VDD, U7.VDDIO, U8.VDD, U8.VDDIO, U9.VDD
- removed net SI4705_!RST: J2.P$5, LED3.A, R33.1, U13.!RST, U15.PTB7/IRQ_3
- removed net SI4705_GPO1: J2.P$19, LED1.A, U13.GPO1
- removed net SI4705_GPO2: J2.P$18, LED2.A, U13.GPO2/!INT
- removed net SI4705_LOUT: J2.P$16, U13.LOUT
- removed net SI4705_LPI: J2.P$15, U13.LPI
- removed net SI4705_ROUT: J2.P$17, U13.ROUT
- removed net SOLAR_VPLUS: D1.+, S1.2
- removed net TPS82740A_CTL/TPS82740A_EN: J3.P$16, U15.PTA9, U6.CTRL, U6.EN
- removed net TPS82740A_LOAD: U6.LOAD
- removed net TPS82740A_VOUT: U14.NC, U6.VOUT
- removed net TPS82740B_CTL/TPS82740B_EN: J3.P$17, U15.PTA12/IRQ_13/LPTMR0_ALT2, U19.CTRL, U19.EN
- removed net TPS82740B_LOAD: U19.LOAD
- removed net TPS82740B_VOUT: U14.NO, U19.VOUT
- removed net TPS82740_DUO_IN: S1.4', U19.VIN, U6.VIN
- removed net TPS82740_VSEL1: J3.P$18, R13.1, U15.PTA5/RTC_CLK_IN, U19.VSEL1, U6.VSEL1
- removed net TPS82740_VSEL2: J3.P$19, R14.1, U15.PTA8, U19.VSEL2, U6.VSEL2
- removed net TPS82740_VSEL3: J3.P$20, R15.1, U15.PTB5/IRQ_12, U19.VSEL3, U6.VSEL3
- removed net TS5A3154_IN: J2.P$7, U14.IN, U15.PTB6/IRQ_2/LPTMR0_ALT3
- removed net TS5A3154_OUT: S1.3, U14.COM
- removed net U20_SO: U20.SDO, U23.SDI
- removed net VBATT: C1.+, C2.+, C4.+, C5.+, C6.+, C7.+, C8.+, C9.+, J2.P$2, J3.P$2, R10.2, R11.2, R27.2, R7.2, S1.1', S1.4, S2.1'
- removed net WARP_VBOOST_IN: C44.1, L3.1, S1.2', S2.3', U21.VIN_DC
- removed net WARP_VBOOST_OUT: S1.1, U21.VBAT
- new net BAT: J1.+
- new net BOOST_EN: S2.1', S2.2'
- new net BOOST_VBAT: S2.2
- new net BOOST_VOUT: S2.3
- new net CHARGE_VOUT: S2.4
- new net FPGA_VS: S1.1', S1.2'
- new net I2C0_SCL/UART_TX: J3.SCL, J4.P$11
- new net I2C0_SDA/UART_RX: J3.SDA, J4.P$12
- new net P10A: J1.P$10
- new net P10B: J2.P$10
- new net P11A: J1.P$11
- new net P11B: J2.P$11
- new net P12A: J1.P$12
- new net P12B: J2.P$12
- new net P13A: J1.P$13
- new net P13B: J2.P$13
- new net P14A: J1.P$14
- new net P14B: J2.P$14
- new net P15A: J1.P$15
- new net P15B: J2.P$15
- new net P16A: J1.P$16
- new net P16B: J2.P$16
- new net P17A: J1.P$17
- new net P17B: J2.P$17
- new net P18A: J1.P$18
- new net P18B: J2.P$18
- new net P19A: J1.P$19
- new net P19B: J2.P$19
- new net P1A: J1.P$1
- new net P1B: J2.P$1
- new net P20A: J1.P$20
- new net P20B: J2.P$20
- new net P2A: J1.P$2
- new net P2B: J2.P$2
- new net P3A: J1.P$3
- new net P3B: J2.P$3
- new net P4A: J1.P$4
- new net P4B: J2.P$4
- new net P5A: J1.P$5
- new net P5B: J2.P$5
- new net P6A: J1.P$6
- new net P6B: J2.P$6
- new net P7A: J1.P$7
- new net P7B: J2.P$7
- new net P8A: J1.P$8
- new net P8B: J2.P$8
- new net P9A: J1.P$9
- new net P9B: J2.P$9
- new net PTA0/SWD_CLK: J1.SWDCLK/TCK
- new net PTA1/RESET_B: J1.!RESET
- new net PTA2/SWD_DIO: J1.SWDIO/TMS
- new net PV_VS: J2.+, J5.P$2
- new net REG_VIN: S2.3', S2.4'
- new net RTC_!INT!/RESET_B: J4.P$7, J5.P$5
- new net SWD_CLK: J4.P$6, J5.P$4
- new net SWD_DIO: J4.P$5, J5.P$3
- new net VCC: J1.VCC, J3.VCC
- new net VS_PRI: J4.P$4, S1.1
- new net VS_SEC: J4.P$3, S1.2
- net GND: now also J1.-, J2.-, J3.GND, J4.P$1, J5.P$1, S2.1; no longer C1.-, C10.2, C11.2, C12.2, C13.2, C14.2, C15.2, C16.2, C17.2, C18.2, C19.2, C2.-, C20.2, C21.2, C22.2, C23.2, C24.2, C25.2, C26.2, C27.2, C28.2, C29.2, C3.2, C30.2, C31.2, C32.2, C33.2, C34.2, C35.2, C36.2, C37.2, C38.2, C39.2, C4.-, C40.2, C42.2, C43.2, C44.2, C45.2, C46.2, C47.2, C48.2, C49.2, C5.-, C50.2, C51.2, C52.2, C53.2, C54.2, C55.2, C56.2, C57.2, C58.2, C59.2, C6.-, C60.2, C61.2, C62.2, C63.2, C64.2, C65.2, C66.2, C67.2, C68.2, C69.2, C7.-, C70.2, C71.2, C72.2, C73.2, C74.2, C75.2, C76.2, C77.2, C78.2, C79.2, C8.-, C80.2, C81.2, C82.2, C9.-, D1.-, J2.P$1, J3.P$1, J6.GND, J7.GND, J7.ID, R1.1, R12.2, R18.1, R2.1, R20.1, R22.1, R3.1, R4.1, R41.2, R42.1, R9.1, S3.B, S3.B', U1.GND@12, U1.GND@13, U1.GND@16, U10.GND, U11.ADDR, U11.GND, U12.GND@1, U12.GND@12, U12.GND@14, U12.GND@20, U13.!SEN, U13.GND@12, U13.GND@PAD, U13.RFGND, U14.EN, U14.GND@C1, U14.GND@D1, U15.VSS, U16.GND@3, U16.GND@8, U16.GND@9, U16.I2C_SA0/SPI4_SDO, U17.!WAKE!, U17.ADDR, U17.GND, U18.AGND, U18.DCNF0, U18.DCNF1, U18.DGND@28, U18.DGND@6, U18.UGND@20, U18.UGND@24, U19.GND, U2.GND1, U2.GND7, U20.VGND, U21.!EN, U21.NC17, U21.NC9, U21.PAD, U21.VSS1, U21.VSS15, U22.GND, U23.VGND, U24.PAD, U25.PAD, U3.CSB3, U3.GNDA, U3.GNDIO, U3.SDO1, U3.SDO2, U4.GND, U5.GND@12, U5.GND@13, U5.I2C_SA0/SPI_SDO, U5.RESERVED@10, U5.RESERVED@11, U5.RESERVED@9, U6.GND, U7.GND@10, U7.GND@5, U8.GND@10, U8.GND@12, U8.GND@5, U8.SA0, U9.GND
- net PAN1326_!SHUTD: now also J4.P$20; no longer J2.P$8, U12.!SHUTD, U15.PTB10
- net SI4705_FMI: now also J5.P$6; no longer J2.P$20, U13.FMI
Other:
- note added: "14: VS_PRI"
- note added: "15: GND"
- note added: "16/7/19"
- note added: "2: GND"
- note added: "3: Signal"
- note added: "5: VS_SEC"
- note added: "6: GND"
- note added: "ADC input replaced by GPIO"
- note added: "AT45DB321F flash chip added"
- note added: "Authored 2015-2019 Phillip Stanley-Marbell Richard Hopper"
- note added: "BOOST"
- note added: "BQ24230 battery charger IC added for LiPo battery"
- note added: "Booster"
- note added: "C"
- note added: "CHARGER"
- note added: "CPX3225A752D supercaps added"
- note added: "Changed to WLP package"
- note added: "Charger"
- note added: "DCPs moved to secondary power supply"
- note added: "DF40 Sockets"
- note added: "DF40 header pin assignments changed"
- note added: "Default pull-ups / downs (sets default voltage to 1.8 V)."
- note added: "EN pin of the BQ25570 can be set"
- note added: "FM ANT"
- note added: "FPGA"
- note added: "FT4222"
- note added: "GPIO lines now powered by external regulator"
- note added: "I2C"
- note added: "IO"
- note added: "Lower loss caps added"
- note added: "MCU"
- note added: "Mechanical switches changed for power control"
- note added: "PV"
- note added: "PV cell wired to header and JST socket"
- note added: "PWR"
- note added: "REG"
- note added: "RF"
- note added: "RTC"
- note added: "RV-8803-C7 RTC IC and coin cell (SR416SW) backup added"
- note added: "Real Time Clock"
- note added: "Regulator"
- note added: "Resistor settings changed for correct charging of supercaps"
- note added: "SENSORS-2"
- note added: "SPI"
- note added: "SWD"
- note added: "Sensors-1"
- note added: "Sensors-2"
- note added: "Settings"
- note added: "Some lines removed from the DF40 header"
- note added: "Split i2c buses for sensors"
- note added: "TOP LEVEL"
- note added: "TPS62172 programmable step-down regulator added"
- note added: "TPS62746DSBGA 1.2 V switching regulator added"
- note added: "Title page"
- note added: "Top Level"
- note added: "Two i2c lines added"
- note added: "Two supply rails VS_PRI (MCU) and VS_SEC (sensors)"
- note added: "UART"
- note added: "USB"
- note added: "USB supply"
- note added: "Update LPS25H footprint"
- note added: "VBAT_OK = 2.2 V"
- note added: "VBAT_OK_HYST = 2.44 V"
- note added: "VBAT_OV = 2.6 V"
- note added: "VBAT_VOUT = 3.8 V"
- note added: "Warp"
- note added: "Warp revision C"
- note removed: "14: vbatt"
- note removed: "15: gnd"
- note removed: "2: Gnd"
- note removed: "3: signal"
- note removed: "5: scaled sensor supply"
- note removed: "6: gnd"
- note removed: "Authored 2015-2018 Phillip Stanley-Marbell"
- note removed: "Warp revision B"
