File: revB/cad/eagle/warp-revC.brd (EAGLE design)
At the start: 48 x 74.3 mm, 183 parts, among them J3 QIIC connector, J4 DF40FC-20DP-0.4V(51), J5 DF40FC-20DP-0.4V(51)

Commit message: Corrected DRC errors, added FT4222 power switch
Parts:
- removed SENSORS-1:U11: GRIDEYE, Grideye:GRIDEYE-AMG88
- removed SENSORS-1:U17: CCS811, SparkFun-Sensors:LGA10
- added FT4222:C3: 4.7uF, SparkFun-Passives:0805
- added FT4222:C4: 0.1uF, SparkFun-Passives:0603-CAP
- added SENSORS-1:U4: GRIDEYE, SparkFun-Sensors:GRIDEYE-AMG88
- added SENSORS-1:U5: CCS811, SparkFun-Sensors:LGA10
- added U$1: CHS-01-SWITCH, CHS_SWITCH:CHS-01_SWITCH
- REG:L2: value (none) -> 2.2uH
- SENSORS-1:R4: value (none) -> 20
Connections:
- net RTC:N$1 renamed RTC:RTC_VDD
- removed net FPGA:IOB_35B_SPI_SS: FPGA:R42.2
- removed net FT4222:GPIO2: FT4222:U18.P$15
- removed net FT4222:GPIO3: FT4222:U18.P$16
- removed net ISL23415_SPI_CS: J4.P$17, MPU:U1.P$20, SENSORS-1:U20.4, SENSORS-1:U23.4
- removed net MPU:N$5: MPU:C37.2
- removed net MPU:N$6: MPU:C36.2
- removed net RF:N$1: RF:C32.2
- removed net RF:N$2: RF:C33.2
- removed net RF:N$3: RF:C35.2
- removed net RF:N$4: RF:C34.2
- removed net RF:SI4705_GPO1: RF:U13.P$19
- removed net RF:SI4705_GPO2: RF:U13.P$18
- removed net SENSORS-1:N$10: SENSORS-1:C12.2
- removed net SENSORS-1:N$11: SENSORS-1:C13.2
- removed net SENSORS-1:N$18: SENSORS-1:C28.2
- removed net SENSORS-1:N$19: SENSORS-1:C29.2
- removed net SENSORS-1:N$20: SENSORS-1:C3.2
- removed net SENSORS-1:N$21: SENSORS-1:C30.2
- removed net SENSORS-1:N$22: SENSORS-1:C40.2
- removed net SENSORS-1:N$23: SENSORS-1:R4.1
- removed net SENSORS-1:N$24: SENSORS-1:C52.2
- removed net SENSORS-1:N$25: SENSORS-1:C50.2
- removed net SENSORS-1:N$27: SENSORS-1:C53.2
- removed net SENSORS-1:N$8: SENSORS-1:C10.2
- removed net SENSORS-1:N$9: SENSORS-1:C11.2
- removed net SENSORS-2:N$11: SENSORS-2:U5.P$5
- removed net SENSORS-2:N$12: SENSORS-2:C15.2, SENSORS-2:C48.2
- removed net SENSORS-2:N$13: SENSORS-2:C23.2
- removed net SENSORS-2:N$14: SENSORS-2:C22.2
- removed net SENSORS-2:N$18: SENSORS-2:C38.2, SENSORS-2:C39.2
- removed net SENSORS-2:N$2: SENSORS-2:C14.2
- removed net SENSORS-2:N$27: SENSORS-2:C16.2
- removed net SENSORS-2:N$28: SENSORS-2:C17.2
- removed net SENSORS-2:N$6: SENSORS-2:C46.2, SENSORS-2:C47.2
- removed net SI4705_!RST!: J4.P$19, MPU:U1.P$14, RF:U13.P$5
- removed net VCC: J3.2
- removed net VS_PRI: FT4222:R23.1, FT4222:R5.2, FT4222:R8.1, FT4222:U18.P$1, FT4222:U18.P$7, J4.P$4, MPU:C36.1, MPU:C37.1, MPU:C51.1, MPU:J1.1, MPU:R10.2, MPU:R11.2, MPU:R7.2, MPU:TP25.TP, MPU:U$1.3, MPU:U$1.6, MPU:U1.P$3, REG:C1.1, REG:L2.2, REG:U1.5, RTC:D3.1, RTC:D3.2, RTC:R40.2, RTC:R6.2, S1.1
- removed net VS_SEC: J4.P$3, REG:U1.6, RF:C32.1, RF:C33.1, RF:C34.1, RF:C35.1, RF:U12.P$10, RF:U12.P$11, RF:U12.P$15, RF:U12.P$22, RF:U13.P$10, RF:U13.P$11, S1.2, SENSORS-1:C10.1, SENSORS-1:C11.1, SENSORS-1:C12.1, SENSORS-1:C13.1, SENSORS-1:C26.1, SENSORS-1:C27.1, SENSORS-1:C28.1, SENSORS-1:C29.1, SENSORS-1:C3.1, SENSORS-1:C30.1, SENSORS-1:C40.1, SENSORS-1:C50.1, SENSORS-1:C52.1, SENSORS-1:C53.1, SENSORS-1:U1.P$1, SENSORS-1:U1.P$14, SENSORS-1:U10.P$1, SENSORS-1:U11.12, SENSORS-1:U11.13, SENSORS-1:U11.9, SENSORS-1:U17.2, SENSORS-1:U17.6, SENSORS-1:U2.2, SENSORS-1:U2.5, SENSORS-1:U2.6, SENSORS-1:U2.8, SENSORS-1:U20.10, SENSORS-1:U20.5, SENSORS-1:U20.8, SENSORS-1:U23.10, SENSORS-1:U23.5, SENSORS-1:U23.8, SENSORS-1:U3.P$13, SENSORS-1:U3.P$3, SENSORS-1:U3.P$7, SENSORS-2:C15.1, SENSORS-2:C16.1, SENSORS-2:C17.1, SENSORS-2:C18.1, SENSORS-2:C19.1, SENSORS-2:C22.1, SENSORS-2:C23.1, SENSORS-2:C24.1, SENSORS-2:C38.1, SENSORS-2:C39.1, SENSORS-2:C46.1, SENSORS-2:C47.1, SENSORS-2:C48.1, SENSORS-2:U16.P$1, SENSORS-2:U16.P$10, SENSORS-2:U16.P$6, SENSORS-2:U4.B1, SENSORS-2:U4.C1, SENSORS-2:U4.D1, SENSORS-2:U5.P$1, SENSORS-2:U5.P$14, SENSORS-2:U5.P$16, SENSORS-2:U7.P$2, SENSORS-2:U7.P$8, SENSORS-2:U8.P$1, SENSORS-2:U8.P$14, SENSORS-2:U9.P$5
- new net FT4222_VCCIO: FT4222:R23.1, FT4222:R5.2, FT4222:R8.1, FT4222:U18.P$1, FT4222:U18.P$7, U$1.1'
- new net ISL23415_SPI_CS/FT4222_GPIO3: FT4222:U18.P$16, J4.P$17, MPU:U1.P$20, SENSORS-1:U20.4, SENSORS-1:U23.4
- new net SENSORS-1:AVDD: SENSORS-1:C41.1, SENSORS-1:U4.10
- new net SENSORS-1:DVDD: SENSORS-1:C40.1, SENSORS-1:U4.12
- new net SENSORS-1:N$1: SENSORS-1:C41.2, SENSORS-1:R4.2
- new net SENSORS-2:CAP: SENSORS-2:C24.1, SENSORS-2:U5.P$14
- new net SI4705_!RST!/FT4222_GPIO2: FT4222:U18.P$15, J4.P$19, MPU:U1.P$14, RF:U13.P$5
- new net VS1: J4.P$4, MPU:C36.1, MPU:C37.1, MPU:C51.1, MPU:J1.1, MPU:R10.2, MPU:R11.2, MPU:R7.2, MPU:TP25.TP, MPU:U$1.3, MPU:U$1.6, MPU:U1.P$3, REG:C1.1, REG:L2.2, REG:U1.5, RTC:D3.1, RTC:D3.2, RTC:R40.2, RTC:R6.2, S1.1, U$1.1
- new net VS2: J3.2, J4.P$3, REG:U1.6, RF:C32.1, RF:C33.1, RF:C34.1, RF:C35.1, RF:U12.P$10, RF:U12.P$11, RF:U12.P$15, RF:U12.P$22, RF:U13.P$10, RF:U13.P$11, S1.2, SENSORS-1:C10.1, SENSORS-1:C11.1, SENSORS-1:C12.1, SENSORS-1:C13.1, SENSORS-1:C26.1, SENSORS-1:C27.1, SENSORS-1:C28.1, SENSORS-1:C29.1, SENSORS-1:C3.1, SENSORS-1:C30.1, SENSORS-1:C50.1, SENSORS-1:C52.1, SENSORS-1:C53.1, SENSORS-1:U1.P$1, SENSORS-1:U1.P$14, SENSORS-1:U10.P$1, SENSORS-1:U2.2, SENSORS-1:U2.5, SENSORS-1:U2.6, SENSORS-1:U2.8, SENSORS-1:U20.10, SENSORS-1:U20.5, SENSORS-1:U20.8, SENSORS-1:U23.10, SENSORS-1:U23.5, SENSORS-1:U23.8, SENSORS-1:U3.P$13, SENSORS-1:U3.P$3, SENSORS-1:U3.P$7, SENSORS-1:U4.13, SENSORS-1:U4.9, SENSORS-1:U5.2, SENSORS-1:U5.6, SENSORS-2:C15.1, SENSORS-2:C16.1, SENSORS-2:C17.1, SENSORS-2:C18.1, SENSORS-2:C19.1, SENSORS-2:C22.1, SENSORS-2:C23.1, SENSORS-2:C38.1, SENSORS-2:C39.1, SENSORS-2:C46.1, SENSORS-2:C47.1, SENSORS-2:C48.1, SENSORS-2:U16.P$1, SENSORS-2:U16.P$10, SENSORS-2:U16.P$6, SENSORS-2:U4.B1, SENSORS-2:U4.C1, SENSORS-2:U4.D1, SENSORS-2:U5.P$1, SENSORS-2:U5.P$16, SENSORS-2:U5.P$5, SENSORS-2:U7.P$2, SENSORS-2:U7.P$8, SENSORS-2:U8.P$1, SENSORS-2:U8.P$14, SENSORS-2:U9.P$5
- net CHARGE_VOUT: now also CHARGER:U$1.5
- net FPGA_CS: now also FPGA:R42.2
- net FT4222:FT4222_VOUT3V3: now also FT4222:C3.1, FT4222:C4.1
- net GND: now also FT4222:C3.2, FT4222:C4.2, MPU:C36.2, MPU:C37.2, RF:C32.2, RF:C33.2, RF:C34.2, RF:C35.2, SENSORS-1:C10.2, SENSORS-1:C11.2, SENSORS-1:C12.2, SENSORS-1:C13.2, SENSORS-1:C28.2, SENSORS-1:C29.2, SENSORS-1:C3.2, SENSORS-1:C30.2, SENSORS-1:C40.2, SENSORS-1:C50.2, SENSORS-1:C52.2, SENSORS-1:C53.2, SENSORS-1:R4.1, SENSORS-1:U4.5, SENSORS-1:U4.6, SENSORS-1:U5.1, SENSORS-1:U5.7, SENSORS-1:U5.EP, SENSORS-2:C14.2, SENSORS-2:C15.2, SENSORS-2:C16.2, SENSORS-2:C17.2, SENSORS-2:C22.2, SENSORS-2:C23.2, SENSORS-2:C38.2, SENSORS-2:C39.2, SENSORS-2:C46.2, SENSORS-2:C47.2, SENSORS-2:C48.2; no longer SENSORS-1:C41.1, SENSORS-1:C41.2, SENSORS-1:R4.2, SENSORS-1:U11.10, SENSORS-1:U11.5, SENSORS-1:U11.6, SENSORS-1:U17.1, SENSORS-1:U17.7, SENSORS-1:U17.EP
- net I2C1_SCL: now also SENSORS-1:U4.3, SENSORS-1:U5.10; no longer SENSORS-1:U11.3, SENSORS-1:U17.10
- net I2C1_SDA: now also SENSORS-1:U4.2, SENSORS-1:U5.9; no longer SENSORS-1:U11.2, SENSORS-1:U17.9
- net SENSORS-1:N$7: now also SENSORS-1:U5.4, SENSORS-1:U5.5; no longer SENSORS-1:U17.4, SENSORS-1:U17.5
Routing:
- added copper zone on layer 1, net BOOST_VOUT
- added copper zone on layer 14, net BOOST_VOUT
- added copper zone on layer 15, net BOOST_VOUT
- added copper zone on layer 16, net BOOST_VOUT
- added copper zone on layer 2, net BOOST_VOUT
- added copper zone on layer 3, net BOOST_VOUT
- added copper zone on layer 4, net BOOST_VOUT
- added copper zone on layer 5, net BOOST_VOUT
- added copper zone on layer 6, net BOOST_VOUT
- added copper zone on layer 7, net BOOST_VOUT
- removed copper zone on layer 1, net BOOST_VIN
- removed copper zone on layer 14, net BOOST_VIN
- removed copper zone on layer 15, net BOOST_VIN
- removed copper zone on layer 16, net BOOST_VIN
- removed copper zone on layer 2, net BOOST_VIN
- removed copper zone on layer 3, net BOOST_VIN
- removed copper zone on layer 4, net BOOST_VIN
- removed copper zone on layer 5, net BOOST_VIN
- removed copper zone on layer 6, net BOOST_VIN
- removed copper zone on layer 7, net BOOST_VIN

Commit message: Layout of charger, boost, reg
Parts:
- removed BOOST:C1, BOOST:C2, BOOST:C4, BOOST:C5, BOOST:C6, BOOST:C7, BOOST:C8, BOOST:C9: CPX3225A7552D, CPX3225A752D:CPX3225A752D
- removed BOOST:C42, BOOST:C44, CHARGER:C2, CHARGER:C3: 4.7uF, SparkFun-Passives:0805
- removed BOOST:C43: 0.1uF, SparkFun-Passives:0603-CAP
- removed BOOST:C45: 10nF, SparkFun-Passives:0603-CAP
- removed BOOST:C49: 22uF, SparkFun-Passives:0805
- removed BOOST:L2: 22uH, EMCComponents (rev19c):WE-TPC_3816
- removed BOOST:L3: 10uH, EMCComponents (rev19c):WE-TPC_2811/2813_OLD
- removed BOOST:R16: 4.02M, SparkFun-Passives:0402-RES
- removed BOOST:R17: 1.3M, SparkFun-Passives:0402-RES
- removed BOOST:R18: 6.49M, SparkFun-Passives:0402-RES
- removed BOOST:R19: 5.36M, SparkFun-Passives:0402-RES
- removed BOOST:R20: 9.09M, SparkFun-Passives:0402-RES
- removed BOOST:R21: 8.87M, SparkFun-Passives:0402-RES
- removed BOOST:R22: 4.22M, SparkFun-Passives:0402-RES
- removed BOOST:TP1, BOOST:TP2, BOOST:TP3, BOOST:TP4, CHARGER:TP1, CHARGER:TP2: TPSTP06R, testpad:TP06R
- removed BOOST:U21: BQ25570PVQFN, BQ25570:BQ25570
- removed CHARGER:C1: 1uF, SparkFun-Passives:0805
- removed CHARGER:D1, CHARGER:D2: (no value), SparkFun-LED:LED-0603
- removed CHARGER:R1: 2.94k, SparkFun-Passives:0402-RES
- removed CHARGER:R2: 4.32k, SparkFun-Passives:0402-RES
- removed CHARGER:R3: 10k, SparkFun-Passives:0402-RES
- removed CHARGER:R4, CHARGER:R5: 4.7k, SparkFun-Passives:0402-RES
- removed CHARGER:R6: 56.2k, SparkFun-Passives:0402-RES
- removed CHARGER:U$1: BQ24230VQFN, BQ24230:PVQFN-N16
- removed J2: (no value), SparkFun-Connectors:JST-2-SMD
- removed U$1: CHS-01-SWITCH, CHS_SWITCH:CHS-01_SWITCH
- removed USB:J7: ZX62-AB-5PA(31)MICRO-AB-SMT, ZX62-AB-5PA(31):ZX62-AB-5PA(31)
- added BAT:C1: 1uF, SparkFun-Passives:0805
- added BAT:C2, BAT:C3, BST:C42, BST:C44: 4.7uF, SparkFun-Passives:0805
- added BAT:D1, BAT:D2: (no value), SparkFun-LED:LED-0603
- added BAT:R1: 2.94k, SparkFun-Passives:0402-RES
- added BAT:R2: 4.32k, SparkFun-Passives:0402-RES
- added BAT:R3: 10k, SparkFun-Passives:0402-RES
- added BAT:R4, BAT:R5: 4.7k, SparkFun-Passives:0402-RES
- added BAT:R6: 56.2k, SparkFun-Passives:0402-RES
- added BAT:TP1, BAT:TP2, BST:TP1, BST:TP2, BST:TP3, BST:TP4, USB2:TP2: TPSTP06R, testpad:TP06R
- added BAT:U$1: BQ24230VQFN, BQ24230:PVQFN-N16
- added BST:C1, BST:C2, BST:C4, BST:C5, BST:C6, BST:C7, BST:C8, BST:C9: CPX3225A7552D, CPX3225A752D:CPX3225A752D
- added BST:C43: 0.1uF, SparkFun-Passives:0603-CAP
- added BST:C45: 10nF, SparkFun-Passives:0603-CAP
- added BST:C49: 22uF, SparkFun-Passives:0805
- added BST:L2: 22uH, EMCComponents (rev19c):WE-TPC_3816
- added BST:L3: 10uH, EMCComponents (rev19c):WE-TPC_2811/2813_OLD
- added BST:R16: 4.02M, SparkFun-Passives:0402-RES
- added BST:R17: 1.3M, SparkFun-Passives:0402-RES
- added BST:R18: 6.49M, SparkFun-Passives:0402-RES
- added BST:R19: 5.36M, SparkFun-Passives:0402-RES
- added BST:R20: 9.09M, SparkFun-Passives:0402-RES
- added BST:R21: 8.87M, SparkFun-Passives:0402-RES
- added BST:R22: 4.22M, SparkFun-Passives:0402-RES
- added BST:U21: BQ25570PVQFN, BQ25570:BQ25570
- added FPGA:J1: WARP-PADS-24, WARP-PADS:PADS-4X6
- added USB1:J1, USB2:J1: J_USB_MICROAB_HIROSE_ZX62-AB-5PA, j_usb_hirose_zx62-ab-5pa:J_USB_MICROAB_HIROSE_ZX62-AB-5PA
- added USB2:C1: 4.7uF (pol), SparkFun-Passives:0402-CAP
- added USB2:C2: 0.1uF, SparkFun-Passives:0402-CAP
- added USB2:FB2: 600R/1A, SparkFun-Passives:0603
- moved FPGA:C3 1406.7 mm to (58.7, 4.83)
- moved FPGA:C13 1399.2 mm to (58.7, -4.57)
- moved FPGA:C10 1398.7 mm to (58.7, 2.29)
- moved FPGA:C11 1396.6 mm to (58.7, -2.54)
- moved FPGA:C14 1394.4 mm to (58.7, -11.2)
- moved FPGA:C5 1392.6 mm to (61.0, 11.7)
- moved FPGA:C6 1391.4 mm to (69.1, 3.56)
- moved FPGA:C12 1388.9 mm to (58.7, -13.5)
- moved FPGA:D1 1386.1 mm to (64.0, -3.05)
- moved REG:L2 1330.3 mm to (0.76, 18.8), turned to 270 degrees
- moved FPGA:C2 1224.1 mm to (71.9, 5.33)
- moved FPGA:U$1 1218.7 mm to (72.9, 2.29)
- moved FPGA:L1 1218.3 mm to (76.2, 3.56)
- moved S2 1201.1 mm to (17.0, 17.0), turned to 90 degrees
- moved REG:C2 1190.5 mm to (4.32, 19.8), turned to 270 degrees
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- renumbered DF40_SOCKETS:J1 to DF40:J1, DF40_SOCKETS:J2 to DF40:J2, FT4222:C1 to FT:C1, FT4222:C2 to FT:C2, FT4222:C3 to FT:C3, FT4222:C4 to FT:C4, FT4222:C62 to FT:C62, FT4222:C63 to FT:C63, FT4222:C64 to FT:C64, FT4222:C65 to FT:C65, FT4222:R23 to FT:R23, FT4222:R25 to FT:R25, FT4222:R5 to FT:R5, FT4222:R8 to FT:R8, FT4222:R9 to FT:R9, FT4222:U18 to FT:U18, FT4222:Y2 to FT:Y2, SENSORS-1:C10 to SEN1:C10, SENSORS-1:C11 to SEN1:C11, SENSORS-1:C12 to SEN1:C12, SENSORS-1:C13 to SEN1:C13, SENSORS-1:C26 to SEN1:C26, SENSORS-1:C27 to SEN1:C27, SENSORS-1:C28 to SEN1:C28, SENSORS-1:C29 to SEN1:C29, SENSORS-1:C3 to SEN1:C3, SENSORS-1:C30 to SEN1:C30, SENSORS-1:C40 to SEN1:C40, SENSORS-1:C41 to SEN1:C41, SENSORS-1:C50 to SEN1:C50, SENSORS-1:C52 to SEN1:C52, SENSORS-1:C53 to SEN1:C53, SENSORS-1:R4 to SEN1:R4, SENSORS-1:U1 to SEN1:U1, SENSORS-1:U10 to SEN1:U10, SENSORS-1:U2 to SEN1:U2, SENSORS-1:U20 to SEN1:U20, SENSORS-1:U23 to SEN1:U23, SENSORS-1:U3 to SEN1:U3, SENSORS-1:U4 to SEN1:U4, SENSORS-1:U5 to SEN1:U5, SENSORS-2:C14 to SEN2:C14, SENSORS-2:C15 to SEN2:C15, SENSORS-2:C16 to SEN2:C16, SENSORS-2:C17 to SEN2:C17, SENSORS-2:C18 to SEN2:C18, SENSORS-2:C19 to SEN2:C19, SENSORS-2:C20 to SEN2:C20, SENSORS-2:C21 to SEN2:C21, SENSORS-2:C22 to SEN2:C22, SENSORS-2:C23 to SEN2:C23, SENSORS-2:C24 to SEN2:C24, SENSORS-2:C38 to SEN2:C38, SENSORS-2:C39 to SEN2:C39, SENSORS-2:C46 to SEN2:C46, SENSORS-2:C47 to SEN2:C47, SENSORS-2:C48 to SEN2:C48, SENSORS-2:U16 to SEN2:U16, SENSORS-2:U4 to SEN2:U4, SENSORS-2:U5 to SEN2:U5, SENSORS-2:U7 to SEN2:U7, SENSORS-2:U8 to SEN2:U8, SENSORS-2:U9 to SEN2:U9, USB:C61 to USB1:C61, USB:C66 to USB1:C66, USB:FB1 to USB1:FB1, USB:TP1 to USB1:TP1
Connections:
- net DF40_SOCKETS:P10A renamed DF40:P10A
- net DF40_SOCKETS:P10B renamed DF40:P10B
- net DF40_SOCKETS:P11A renamed DF40:P11A
- net DF40_SOCKETS:P11B renamed DF40:P11B
- net DF40_SOCKETS:P12A renamed DF40:P12A
- net DF40_SOCKETS:P12B renamed DF40:P12B
- net DF40_SOCKETS:P13A renamed DF40:P13A
- net DF40_SOCKETS:P13B renamed DF40:P13B
- net DF40_SOCKETS:P14A renamed DF40:P14A
- net DF40_SOCKETS:P14B renamed DF40:P14B
- net DF40_SOCKETS:P15A renamed DF40:P15A
- net DF40_SOCKETS:P15B renamed DF40:P15B
- net DF40_SOCKETS:P16A renamed DF40:P16A
- net DF40_SOCKETS:P16B renamed DF40:P16B
- net DF40_SOCKETS:P17A renamed DF40:P17A
- net DF40_SOCKETS:P17B renamed DF40:P17B
- net DF40_SOCKETS:P18A renamed DF40:P18A
- net DF40_SOCKETS:P18B renamed DF40:P18B
- net DF40_SOCKETS:P19A renamed DF40:P19A
- net DF40_SOCKETS:P19B renamed DF40:P19B
- net DF40_SOCKETS:P1A renamed DF40:P1A
- net DF40_SOCKETS:P1B renamed DF40:P1B
- net DF40_SOCKETS:P20A renamed DF40:P20A
- net DF40_SOCKETS:P20B renamed DF40:P20B
- net DF40_SOCKETS:P2A renamed DF40:P2A
- net DF40_SOCKETS:P2B renamed DF40:P2B
- net DF40_SOCKETS:P3A renamed DF40:P3A
- net DF40_SOCKETS:P3B renamed DF40:P3B
- net DF40_SOCKETS:P4A renamed DF40:P4A
- net DF40_SOCKETS:P4B renamed DF40:P4B
- net DF40_SOCKETS:P5A renamed DF40:P5A
- net DF40_SOCKETS:P5B renamed DF40:P5B
- net DF40_SOCKETS:P6A renamed DF40:P6A
- net DF40_SOCKETS:P6B renamed DF40:P6B
- net DF40_SOCKETS:P7A renamed DF40:P7A
- net DF40_SOCKETS:P7B renamed DF40:P7B
- net DF40_SOCKETS:P8A renamed DF40:P8A
- net DF40_SOCKETS:P8B renamed DF40:P8B
- net DF40_SOCKETS:P9A renamed DF40:P9A
- net DF40_SOCKETS:P9B renamed DF40:P9B
- net FT4222:FT4222_VOUT3V3 renamed FT:FT4222_VOUT3V3
- net FT4222:N$15 renamed FT:N$15
- net FT4222:N$2 renamed FT:N$2
- net FT4222:N$3 renamed FT:N$3
- net FT4222:N$4 renamed FT:N$4
- net FT4222:N$5 renamed FT:N$5
- net FT4222:N$6 renamed FT:N$6
- net FT4222:VPP renamed FT:VPP
- net IOB_13B renamed FPGA:IOB_13B
- net IOT_47A renamed FPGA:IOT_47A
- net SENSORS-1:AVDD renamed SEN1:AVDD
- net SENSORS-1:DVDD renamed SEN1:DVDD
- net SENSORS-1:N$1 renamed SEN1:N$1
- net SENSORS-1:N$7 renamed SEN1:N$7
- net SENSORS-2:CAP renamed SEN2:CAP
- net SENSORS-2:N$1 renamed SEN2:N$1
- net SENSORS-2:N$17 renamed SEN2:N$17
- removed net BOOST:LBOOST: BOOST:L2.2, BOOST:U21.20
- removed net BOOST:LBUCK: BOOST:L3.1, BOOST:U21.16
- removed net BOOST:OK_HYST: BOOST:R17.1, BOOST:R19.2, BOOST:U21.10
- removed net BOOST:OK_PROG: BOOST:R18.2, BOOST:R19.1, BOOST:U21.11
- removed net BOOST:VBAT_OV: BOOST:R16.1, BOOST:R20.2, BOOST:U21.7
- removed net BOOST:VOUT_SET: BOOST:R21.1, BOOST:R22.2, BOOST:U21.12
- removed net BOOST:VRDIV: BOOST:R16.2, BOOST:R17.2, BOOST:R21.2, BOOST:U21.8
- removed net BOOST:VREF_SAMP: BOOST:C45.1, BOOST:U21.4
- removed net BOOST:VSTOR: BOOST:C42.1, BOOST:C43.1, BOOST:TP4.TP, BOOST:U21.19, BOOST:U21.3, BOOST:U21.6
- removed net CHARGER:N$1: CHARGER:R2.2, CHARGER:U$1.16
- removed net CHARGER:N$2: CHARGER:R1.2, CHARGER:U$1.12
- removed net CHARGER:N$3: CHARGER:R4.1, CHARGER:U$1.7
- removed net CHARGER:N$4: CHARGER:R3.2, CHARGER:U$1.1
- removed net CHARGER:N$5: CHARGER:R5.1, CHARGER:U$1.9
- removed net CHARGER:N$6: CHARGER:D1.C, CHARGER:R4.2
- removed net CHARGER:N$7: CHARGER:D2.C, CHARGER:R5.2
- removed net CHARGER:N$8: CHARGER:R6.2, CHARGER:U$1.14
- removed net FT4222_VCCIO: FT:R23.1, FT:R5.2, FT:R8.1, FT:U18.P$1, FT:U18.P$7, U$1.1'
- removed net IOB_12A_G4_CDONE: FPGA:U$7.D3
- removed net IOB_24A: FPGA:U$7.B1
- removed net IOB_25B_G3: FPGA:U$7.F2
- removed net IOB_2A: FPGA:U$7.D5
- removed net IOB_3B_G6: FPGA:U$7.F5
- removed net IOB_9B: FPGA:U$7.E4
- removed net IOT_46B_G0: FPGA:U$7.B3
- removed net N$1: FT:U18.P$23, USB:J7.3
- removed net N$2: FT:U18.P$22, USB:J7.2
- removed net RGB0: FPGA:U$7.A5
- removed net RGB1: FPGA:U$7.B5
- removed net RGB2: FPGA:U$7.C5
- removed net USB:VBUS: USB1:FB1.2, USB:J7.1
- new net BAT:N$1: BAT:R2.2, BAT:U$1.16
- new net BAT:N$2: BAT:R1.2, BAT:U$1.12
- new net BAT:N$3: BAT:R4.1, BAT:U$1.7
- new net BAT:N$4: BAT:R3.2, BAT:U$1.1
- new net BAT:N$5: BAT:R5.1, BAT:U$1.9
- new net BAT:N$6: BAT:D1.C, BAT:R4.2
- new net BAT:N$7: BAT:D2.C, BAT:R5.2
- new net BAT:N$8: BAT:R6.2, BAT:U$1.14
- new net BST:LBOOST: BST:L2.2, BST:U21.20
- new net BST:LBUCK: BST:L3.1, BST:U21.16
- new net BST:OK_HYST: BST:R17.1, BST:R19.2, BST:U21.10
- new net BST:OK_PROG: BST:R18.2, BST:R19.1, BST:U21.11
- new net BST:VBAT_OV: BST:R16.1, BST:R20.2, BST:U21.7
- new net BST:VOUT_SET: BST:R21.1, BST:R22.2, BST:U21.12
- new net BST:VRDIV: BST:R16.2, BST:R17.2, BST:R21.2, BST:U21.8
- new net BST:VREF_SAMP: BST:C45.1, BST:U21.4
- new net BST:VSTOR: BST:C42.1, BST:C43.1, BST:TP4.TP, BST:U21.19, BST:U21.3, BST:U21.6
- new net FPGA:IC21_SDA: FPGA:J1.18
- new net FPGA:IOB13B: FPGA:J1.11
- new net FPGA:IOB_12A_G4_CDONE: FPGA:J1.20, FPGA:U$7.D3
- new net FPGA:IOB_24A: FPGA:J1.7, FPGA:U$7.B1
- new net FPGA:IOB_25B_G3: FPGA:J1.17, FPGA:U$7.F2
- new net FPGA:IOB_2A: FPGA:J1.21, FPGA:U$7.D5
- new net FPGA:IOB_3B_G6: FPGA:J1.23, FPGA:U$7.F5
- new net FPGA:IOB_9B: FPGA:J1.16, FPGA:U$7.E4
- new net FPGA:IOT47A: FPGA:J1.4
- new net FPGA:IOT_46B_G0: FPGA:J1.8, FPGA:U$7.B3
- new net FPGA:N$3: FPGA:J1.24
- new net FPGA:RGB0: FPGA:J1.5, FPGA:U$7.A5
- new net FPGA:RGB1: FPGA:J1.10, FPGA:U$7.B5
- new net FPGA:RGB2: FPGA:J1.15, FPGA:U$7.C5
- new net USB1:VBUS: USB1:FB1.2, USB1:J1.P$1
- new net USB2:DM: USB2:J1.P$2
- new net USB2:DP: USB2:J1.P$3
- new net USB2:VBUS: USB2:FB2.2, USB2:J1.P$1
- new net USB_DM: FT:U18.P$22, USB1:J1.P$2
- new net USB_DP: FT:U18.P$23, USB1:J1.P$3
- net BAT: now also BAT:C3.1, BAT:TP1.TP, BAT:U$1.2, BAT:U$1.3; no longer CHARGER:C3.1, CHARGER:TP1.TP, CHARGER:U$1.2, CHARGER:U$1.3
- net BOOST_EN: now also BST:U21.5; no longer BOOST:U21.5
- net BOOST_VBAT: now also BST:C1.+, BST:C2.+, BST:C4.+, BST:C5.+, BST:C6.+, BST:C7.+, BST:C8.+, BST:C9.+, BST:TP3.TP, BST:U21.18; no longer BOOST:C1.+, BOOST:C2.+, BOOST:C4.+, BOOST:C5.+, BOOST:C6.+, BOOST:C7.+, BOOST:C8.+, BOOST:C9.+, BOOST:TP3.TP, BOOST:U21.18
- net BOOST_VOUT: now also BST:C49.1, BST:L3.2, BST:TP2.TP, BST:U21.14; no longer BOOST:C49.1, BOOST:L3.2, BOOST:TP2.TP, BOOST:U21.14
- net CHARGE_VOUT: now also BAT:C2.1, BAT:D1.A, BAT:D2.A, BAT:TP2.TP, BAT:U$1.10, BAT:U$1.11, BAT:U$1.5; no longer CHARGER:C2.1, CHARGER:D1.A, CHARGER:D2.A, CHARGER:TP2.TP, CHARGER:U$1.10, CHARGER:U$1.11, CHARGER:U$1.5
- net FPGA:IOB_0A: now also FPGA:J1.22
- net FPGA_CS: now also FPGA:J1.13
- net FPGA_VS: now also FPGA:J1.3
- net GND: now also BAT:C1.2, BAT:C2.2, BAT:C3.2, BAT:R1.1, BAT:R2.1, BAT:R3.1, BAT:R6.1, BAT:U$1.15, BAT:U$1.4, BAT:U$1.6, BAT:U$1.8, BAT:U$1.EP, BST:C1.-, BST:C2.-, BST:C4.-, BST:C42.2, BST:C43.2, BST:C44.2, BST:C45.2, BST:C49.2, BST:C5.-, BST:C6.-, BST:C7.-, BST:C8.-, BST:C9.-, BST:R18.1, BST:R20.1, BST:R22.1, BST:U21.1, BST:U21.15, BST:U21.17, BST:U21.21, BST:U21.9, FPGA:J1.9, USB1:J1.P$5, USB1:J1.SHIELD1, USB1:J1.SHIELD2, USB1:J1.SHIELD3, USB1:J1.SHIELD4, USB2:C1.2, USB2:C2.2, USB2:J1.P$5, USB2:J1.SHIELD1, USB2:J1.SHIELD2, USB2:J1.SHIELD3, USB2:J1.SHIELD4; no longer BOOST:C1.-, BOOST:C2.-, BOOST:C4.-, BOOST:C42.2, BOOST:C43.2, BOOST:C44.2, BOOST:C45.2, BOOST:C49.2, BOOST:C5.-, BOOST:C6.-, BOOST:C7.-, BOOST:C8.-, BOOST:C9.-, BOOST:R18.1, BOOST:R20.1, BOOST:R22.1, BOOST:U21.1, BOOST:U21.15, BOOST:U21.17, BOOST:U21.21, BOOST:U21.9, CHARGER:C1.2, CHARGER:C2.2, CHARGER:C3.2, CHARGER:R1.1, CHARGER:R2.1, CHARGER:R3.1, CHARGER:R6.1, CHARGER:U$1.15, CHARGER:U$1.4, CHARGER:U$1.6, CHARGER:U$1.8, CHARGER:U$1.EP, J2.1, USB:J7.4, USB:J7.5
- net I2C1_SCL: now also FPGA:J1.14
- net I2C2_SCL: now also FPGA:J1.2
- net I2C2_SDA: now also FPGA:J1.1
- net PV_VS: now also BST:C44.1, BST:L2.1, BST:TP1.TP, BST:U21.2, J5.P$8; no longer BOOST:C44.1, BOOST:L2.1, BOOST:TP1.TP, BOOST:U21.2, J2.2, J5.P$2
- net RTC_!INT!/RESET_B: now also J5.P$7; no longer J5.P$5
- net SI4705_FMI: no longer J5.P$6
- net SPI_MISO/UART_RTS: now also FPGA:J1.12
- net SPI_MOSI/UART_CTS: now also FPGA:J1.6
- net SPI_SCK: now also FPGA:J1.19
- net SWD_CLK: now also J5.P$6; no longer J5.P$4
- net SWD_DIO: now also J5.P$5; no longer J5.P$3
- net USB_5V: now also BAT:C1.1, BAT:U$1.13, J5.P$2, USB2:C1.1, USB2:C2.1, USB2:FB2.1, USB2:TP2.TP; no longer CHARGER:C1.1, CHARGER:U$1.13
- net VS1: now also FT:R23.1, FT:R5.2, FT:R8.1, FT:U18.P$1, FT:U18.P$7, J5.P$4; no longer U$1.1
- net VS2: now also J5.P$3
Routing:
- net BOOST_VBAT: track 2.27 -> 48.5 mm
- net CHARGE_VOUT: track 0.00 -> 15.1 mm
- net BOOST_EN: track 0.00 -> 13.8 mm, vias 0 -> 2
- net BOOST_VOUT: track 0.00 -> 11.2 mm
- net BST:VRDIV: track 0.00 -> 11.0 mm, vias 0 -> 2
- net REG_VIN: track 0.00 -> 9.63 mm
- net PV_VS: track 0.00 -> 6.97 mm
- net USB_5V: track 0.00 -> 6.81 mm
- net REG:SW: track 0.00 -> 6.26 mm
- net VS1: track 0.00 -> 5.97 mm, vias 0 -> 1
- net BST:VOUT_SET: track 0.00 -> 5.93 mm
- net BST:VSTOR: track 0.00 -> 5.82 mm
- net BST:LBOOST: track 0.00 -> 5.57 mm
- net BST:VREF_SAMP: track 0.00 -> 5.49 mm
- net BST:OK_HYST: track 0.00 -> 5.44 mm
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- added copper zone on layer 5, net VS1
- added copper zone on layer 7, net VSS2
- removed copper zone on layer 14, net BOOST_VBAT
- removed copper zone on layer 1, net BOOST_VOUT
- removed copper zone on layer 14, net BOOST_VOUT
- removed copper zone on layer 15, net BOOST_VOUT
- removed copper zone on layer 16, net BOOST_VOUT
- removed copper zone on layer 2, net BOOST_VOUT
- removed copper zone on layer 3, net BOOST_VOUT
- removed copper zone on layer 5, net BOOST_VOUT
- removed copper zone on layer 7, net BOOST_VOUT
- removed copper zone on layer 1, net GND
- removed copper zone on layer 7, net ICE40_VCCIO
- removed copper zone on layer 5, net SCALED_SENSOR_SUPPLY
Other:
- board text removed: "Warp Rev. B, Bottom"

Commit message: FPGA layout
Parts:
- removed FPGA:C10: 0.1uF, SparkFun-Passives:0603-CAP
- removed FPGA:C14, FPGA:C3: 1uF, SparkFun-Passives:0805
- removed FPGA:C4: 10nF, SparkFun-Passives:0402-CAP
- removed FPGA:D1: BLUE, SparkFun-LED:LED-0603
- removed FPGA:L1: 2.2uH, WURTH-744025002:WURTH-744025002
- removed FPGA:R41: 4.7k, SparkFun-Passives:0402-RES
- removed FPGA:R42: DNP, SparkFun-Passives:0402-RES
- added FPGA:C1: 1uF, SparkFun-Passives:0805
- FPGA:C2: value 4.7uF -> 1uF
- FPGA:J1: value WARP-PADS-24 -> WARP-PADS-22; device WARP-PADS:PADS-4X6 -> WARP-PADS:PADS-22
- FPGA:U$1: value TPS62746DSBGA(8) -> MCP1811AT-012/TTSOT-23-3; device TPS62746:DSBGA -> MCP1811AT-012:TT:SOT23-3
- moved DF40:J2 1527.1 mm to (122.9, 64.5)
- moved DF40:J1 1500.7 mm to (74.8, 64.4)
- moved MPU:U1 1414.2 mm to (22.2, 20.3)
- moved FD1 1389.1 mm to (-72.9, 10.8)
- moved FD2 1389.1 mm to (-73.7, 5.46)
- moved FD3 1389.1 mm to (-73.2, 9.02)
- moved FD5 1389.1 mm to (-73.4, 7.24)
- moved FD4 1389.1 mm to (-73.9, 3.68)
- moved SEN1:U4 1375.6 mm to (-98.7, -24.0)
- moved SEN1:U5 1375.6 mm to (-103.5, -15.1)
- moved MPU:U$1 1326.2 mm to (28.6, 19.9), turned to 90 degrees
- moved J5 1306.2 mm to (35.7, 14.4), turned to 270 degrees
- moved J4 1306.1 mm to (35.7, 21.8), turned to 270 degrees
- moved FT:C1 1294.6 mm to (6.22, -27.7)
- moved FT:C2 1294.6 mm to (6.22, -31.2)
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Connections:
- removed net FPGA:IC21_SDA: FPGA:J1.18
- removed net FPGA:IOB13B: FPGA:J1.11
- removed net FPGA:IOB_12A_G4_CDONE: FPGA:J1.20, FPGA:U$7.D3
- removed net FPGA:IOB_25B_G3: FPGA:J1.17, FPGA:U$7.F2
- removed net FPGA:IOT47A: FPGA:J1.4
- removed net FPGA:N$1: FPGA:D1.C, FPGA:R41.1
- removed net FPGA:N$2: FPGA:L1.1, FPGA:U$1.A1
- removed net FPGA:N$3: FPGA:J1.24
- net FPGA:IOB_0A: now also FPGA:J1.6; no longer FPGA:D1.A, FPGA:J1.22
- net FPGA:IOB_13B: now also FPGA:J1.16
- net FPGA:IOB_24A: now also FPGA:J1.9; no longer FPGA:J1.7
- net FPGA:IOB_2A: now also FPGA:J1.17; no longer FPGA:J1.21
- net FPGA:IOB_3B_G6: now also FPGA:J1.11; no longer FPGA:J1.23
- net FPGA:IOB_9B: now also FPGA:J1.22; no longer FPGA:J1.16
- net FPGA:IOT_46B_G0: now also FPGA:J1.13; no longer FPGA:J1.8
- net FPGA:IOT_47A: now also FPGA:J1.2
- net FPGA:RGB0: now also FPGA:J1.7; no longer FPGA:J1.5
- net FPGA:RGB1: now also FPGA:J1.12; no longer FPGA:J1.10
- net FPGA:RGB2: now also FPGA:J1.1; no longer FPGA:J1.15
- net FPGA:VCC_1V2: now also FPGA:C12.1, FPGA:C2.1, FPGA:C79.1, FPGA:U$1.1; no longer FPGA:L1.2, FPGA:U$1.C2
- net FPGA_CS: now also FPGA:J1.20; no longer FPGA:J1.13, FPGA:R42.2
- net FPGA_VS: now also FPGA:J1.8; no longer FPGA:C10.1, FPGA:C12.1, FPGA:C14.1, FPGA:C3.1, FPGA:C4.1, FPGA:C79.1, FPGA:J1.3, FPGA:U$1.B1
- net GND: now also FPGA:C1.2, FPGA:J1.18, FPGA:J1.19, FPGA:U$1.3; no longer FPGA:C10.2, FPGA:C14.2, FPGA:C3.2, FPGA:C4.2, FPGA:J1.9, FPGA:R41.2, FPGA:R42.1, FPGA:U$1.B2, FPGA:U$1.C1
- net I2C1_SCL: now also FPGA:J1.21, FPGA:U$7.F2; no longer FPGA:J1.14, FPGA:U$7.C3
- net I2C1_SDA: now also FPGA:J1.5
- net I2C2_SCL: now also FPGA:J1.3; no longer FPGA:J1.2
- net I2C2_SDA: now also FPGA:J1.14; no longer FPGA:J1.1
- net SPI_MISO/UART_RTS: now also FPGA:J1.10; no longer FPGA:J1.12
- net SPI_MOSI/UART_CTS: now also FPGA:J1.15; no longer FPGA:J1.6
- net SPI_SCK: now also FPGA:J1.4; no longer FPGA:J1.19
- net USB_5V: now also FPGA:C1.1, FPGA:U$1.2; no longer FPGA:C2.1, FPGA:U$1.A2
Routing:
- net FPGA_VS: track 0.00 -> 48.1 mm, vias 0 -> 4
- net FPGA:ICE40_VCC_PLL: track 0.00 -> 30.7 mm, vias 0 -> 2
- net FPGA:IOB_9B: track 0.00 -> 23.9 mm, vias 0 -> 1
- net FPGA:IOB_13B: track 0.00 -> 19.1 mm, vias 0 -> 1
- net FPGA:VCC_1V2: track 0.25 -> 18.5 mm, vias 0 -> 3
- net FPGA:IOT_46B_G0: track 0.00 -> 17.2 mm, vias 0 -> 1
- net FPGA:IOB_2A: track 0.00 -> 13.9 mm
- net FPGA:RGB1: track 0.00 -> 12.2 mm
- net BOOST_VBAT: track 48.5 -> 37.3 mm
- net FPGA:RGB2: track 0.01 -> 10.9 mm
- net FPGA:IOB_0A: track 0.00 -> 9.63 mm
- net I2C1_SCL: track 0.00 -> 9.26 mm
- net FPGA:RGB0: track 0.00 -> 9.03 mm
- net FPGA:IOB_3B_G6: track 0.00 -> 8.39 mm
- net BOOST_VOUT: track 11.2 -> 3.32 mm
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
Commit message: Top layout 70% complete
Parts:
- removed BST:TP4, MPU:TP25, RTC:TP12: TPSTP06R, testpad:TP06R
- removed FPGA:J1: WARP-PADS-22, WARP-PADS:PADS-22
- removed J5: DF40FC-20DP-0.4V(51), DF40FC-20DP-0.4V(51):DF40C-20DP-0.4V(51)
- removed RTC:D2: 250mA/100V, SparkFun-DiscreteSemi:SOD-323
- removed RTC:D3: BAS70-05, diode:SOT23
- removed RTC:U$6: ML414_BATTERY_CONTACT, ML414:ML414
- removed S2: CHS-04_SWITCH, CHS_SWITCH:CHS-04_SWITCH
- added J2: (no value), SparkFun-Connectors:JST-2-SMD
- added S3: CHS-02_SWITCH, CHS_SWITCH:CHS-02_SWITCH
- moved USB1:TP1 141.6 mm to (11.6, 68.1)
- moved USB1:FB1 137.9 mm to (7.87, 67.4)
- moved SEN1:U2 134.6 mm to (23.0, -43.1)
- moved SEN1:C10 134.6 mm to (31.6, -45.0)
- moved SEN1:C11 134.6 mm to (23.6, -18.2)
- moved SEN1:C12 134.6 mm to (23.6, -21.2)
- moved SEN1:C13 134.6 mm to (23.6, -24.3)
- moved SEN1:C26 134.6 mm to (23.6, -27.3)
- moved SEN1:C27 134.6 mm to (23.6, -30.4)
- moved SEN1:C28 134.6 mm to (23.6, -33.4)
- moved SEN1:C29 134.6 mm to (23.6, -36.4)
- moved SEN1:C3 134.6 mm to (16.3, -26.3)
- moved SEN1:C30 134.6 mm to (16.3, -29.3)
- moved SEN1:C40 134.6 mm to (16.3, -32.4)
- moved SEN1:C41 134.6 mm to (16.3, -35.4)
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Connections:
- removed net BOOST_EN: BST:U21.5, S2.1', S2.2'
- removed net FPGA:IOB_0A: FPGA:J1.6, FPGA:U$7.E5
- removed net FPGA:IOB_13B: FPGA:J1.16, FPGA:U$7.E3
- removed net FPGA:IOB_24A: FPGA:J1.9, FPGA:U$7.B1
- removed net FPGA:IOB_2A: FPGA:J1.17, FPGA:U$7.D5
- removed net FPGA:IOB_3B_G6: FPGA:J1.11, FPGA:U$7.F5
- removed net FPGA:IOB_9B: FPGA:J1.22, FPGA:U$7.E4
- removed net FPGA:IOT_46B_G0: FPGA:J1.13, FPGA:U$7.B3
- removed net FPGA:IOT_47A: FPGA:J1.2, FPGA:U$7.A4
- removed net FPGA:RGB0: FPGA:J1.7, FPGA:U$7.A5
- removed net FPGA:RGB1: FPGA:J1.12, FPGA:U$7.B5
- removed net FPGA:RGB2: FPGA:J1.1, FPGA:U$7.C5
- removed net RTC:RTC_VDD: RTC:C1.1, RTC:D2.C, RTC:D3.3, RTC:U$5.3
- removed net RTC:VBB: RTC:D2.A, RTC:TP12.TP, RTC:U$6.1, RTC:U$6.3
- net BOOST_VBAT: no longer S2.2
- net BOOST_VOUT: now also S3.1; no longer S2.3
- net BST:VSTOR: no longer BST:TP4.TP
- net CHARGE_VOUT: now also S3.2; no longer S2.4
- net FPGA:ICE40_VCC_PLL: now also FPGA:U$7.B1
- net FPGA_CS: no longer FPGA:J1.20
- net FPGA_VS: now also FPGA:U$7.C5; no longer FPGA:J1.8
- net GND: now also BST:U21.5, FPGA:U$7.F2, J2.1; no longer FPGA:J1.18, FPGA:J1.19, J5.P$1, RTC:U$6.2, S2.1
- net I2C1_SCL: now also FPGA:U$7.A4; no longer FPGA:J1.21, FPGA:U$7.F2
- net I2C1_SDA: no longer FPGA:J1.5
- net I2C2_SCL: no longer FPGA:J1.3
- net I2C2_SDA: no longer FPGA:J1.14
- net PV_VS: now also J2.2, J4.P$4; no longer J5.P$8
- net REG_VIN: now also FPGA:C1.1, FPGA:U$1.2, S3.1', S3.2'; no longer S2.3', S2.4'
- net RTC_!INT!/RESET_B: no longer J5.P$7
- net SPI_MISO/UART_RTS: no longer FPGA:J1.10
- net SPI_MOSI/UART_CTS: no longer FPGA:J1.15
- net SPI_SCK: no longer FPGA:J1.4
- net SWD_CLK: no longer J5.P$6
- net SWD_DIO: no longer J5.P$5
- net USB_5V: no longer FPGA:C1.1, FPGA:U$1.2, J5.P$2
- net VS1: now also RTC:C1.1, RTC:U$5.3; no longer J4.P$4, J5.P$4, MPU:TP25.TP, RTC:D3.1, RTC:D3.2
- net VS2: no longer J5.P$3
Routing:
- net FPGA_VS: track 48.1 -> 17.9 mm, vias 4 -> 2
- net BOOST_VOUT: track 3.32 -> 29.4 mm, vias 0 -> 2
- net FPGA:IOB_9B: track 23.9 -> 0.00 mm, vias 1 -> 0
- net FPGA:ICE40_VCC_PLL: track 30.7 -> 6.98 mm, vias 2 -> 0
- net REG_VSEL1: track 0.00 -> 19.5 mm, vias 0 -> 2
- net FPGA:IOB_13B: track 19.1 -> 0.00 mm, vias 1 -> 0
- net FPGA:IOT_46B_G0: track 17.2 -> 0.00 mm, vias 1 -> 0
- net FPGA:IOB_2A: track 13.9 -> 0.00 mm
- net FPGA:RGB1: track 12.2 -> 0.00 mm
- net BAT: track 2.93 -> 15.1 mm, vias 0 -> 1
- net VS1: track 5.97 -> 17.7 mm, vias 1 -> 2
- net RTC_!INT!/RESET_B: track 0.00 -> 11.3 mm
- net FPGA:RGB2: track 10.9 -> 0.00 mm
- net FPGA:IOB_0A: track 9.63 -> 0.00 mm
- net I2C1_SCL: track 9.26 -> 0.00 mm
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- added copper zone on layer 1, net BAT
- added copper zone on layer 16, net BAT
- added copper zone on layer 1, net CHARGE_VOUT
- added copper zone on layer 1, net GND
- added copper zone on layer 14, net GND
- added copper zone on layer 3, net GND
- added copper zone on layer 7, net GND
- added copper zone on layer 1, net REG_VIN
- added copper zone on layer 1, net USB2:VBUS
- added copper zone on layer 1, net USB_5V
- added copper zone on layer 1, net VS1
- added copper zone on layer 4, net VS1
- added copper zone on layer 1, net VS2
- added copper zone on layer 16, net VS2
- removed copper zone on layer 4, net BOOST_VOUT
- removed copper zone on layer 6, net BOOST_VOUT
- removed copper zone on layer 7, net VSS2
Other:
- board size 48 x 74.3 mm -> 46.7 x 72.8 mm
- board text added: "REV C"
- board text removed: "REV B"
- board text removed: "SSSPLY"
- board text removed: "VBOOSTIN"
