File: revB/cad/eagle/warp-revC.sch (EAGLE design)
At the start: 12 parts, among them J3 QIIC connector, J4 DF40FC-20DP-0.4V(51), J5 DF40FC-20DP-0.4V(51)

Commit message: Corrected DRC errors, added FT4222 power switch
Parts:
- added U$1: CHS-01-SWITCH, CHS_SWITCH:CHS-01-SWITCH
Connections:
- net ISL23415_SPI_CS renamed ISL23415_SPI_CS/FT4222_GPIO3
- net SI4705_!RST! renamed SI4705_!RST!/FT4222_GPIO2
- removed net VS_PRI: J4.P$4, S1.1
- removed net VS_SEC: J4.P$3, S1.2
- new net AT45DB321F_SPI_CS: U$1.!CS!
- new net EN: U$1.EN
- new net FT4222_VCCIO: U$1.1'
- new net IN: U$1.IN
- new net N$1: U$1.ISET
- new net N$2: U$1.ILIM, U$1.SW
- new net N$3: U$1.!PGOOD!
- new net N$4: U$1.!WP!, U$1.TS
- new net N$5: U$1.!CHG!
- new net N$8: U$1.TMR
- new net OUT: U$1.EN2, U$1.OUT
- new net SPI_MISO: U$1.SO
- new net SPI_MOSI: U$1.SI
- new net VCC_1V2: U$1.VOS
- new net VREG: U$1.VIN
- new net VS1: J4.P$4, S1.1, U$1.1
- new net VS2: J3.VCC, J4.P$3, S1.2
- net BAT: now also U$1.BAT
- net GND: now also U$1.!CE!, U$1.EN1, U$1.GND, U$1.TD, U$1.VSEL, U$1.VSS
- net SPI_SCK: now also U$1.SCK
- net VCC: now also U$1.!RST!, U$1.VCC; no longer J3.VCC
Other:
- note added: "19/7/19"
- note added: "Battery JST socket"
- note added: "External sensor socket"
- note added: "FT4222 pwr break"
- note added: "Header sockets"
- note added: "PV cell JST socket"
- note added: "Power source switching"
- note added: "Primary and secondary supply rails (VS1, VS2)"
- note added: "Sockets to break out lines"
- note added: "Supply select for FPGA"
- note added: "Switch added to break supply (for power save mode)"
- note removed: "16/7/19"
- note removed: "Two supply rails VS_PRI (MCU) and VS_SEC (sensors)"
- moved on the sheet: J1, J2, J4, J5

Commit message: Layout of charger, boost, reg
Parts:
- removed J2: (no value), SparkFun-Connectors:JST_2MM_MALE
- removed U$1: CHS-01-SWITCH, CHS_SWITCH:CHS-01-SWITCH
Connections:
- removed net AT45DB321F_SPI_CS: U$1.!CS!
- removed net EN: U$1.EN
- removed net FT4222_VCCIO: U$1.1'
- removed net IN: U$1.IN
- removed net N$1: U$1.ISET
- removed net N$2: U$1.ILIM, U$1.SW
- removed net N$4: U$1.!WP!, U$1.TS
- removed net N$5: U$1.!CHG!
- removed net N$8: U$1.TMR
- removed net OUT: U$1.EN2, U$1.OUT
- removed net P10B: J2.P$10
- removed net P11B: J2.P$11
- removed net P12B: J2.P$12
- removed net P13B: J2.P$13
- removed net P14B: J2.P$14
- removed net P15B: J2.P$15
- removed net P16B: J2.P$16
- removed net P17B: J2.P$17
- removed net P18B: J2.P$18
- removed net P19B: J2.P$19
- removed net P1B: J2.P$1
- removed net P20B: J2.P$20
- removed net P2B: J2.P$2
- removed net P3B: J2.P$3
- removed net P4B: J2.P$4
- removed net P5B: J2.P$5
- removed net P6B: J2.P$6
- removed net P7B: J2.P$7
- removed net P8B: J2.P$8
- removed net P9B: J2.P$9
- removed net SI4705_FMI: J5.P$6
- removed net VCC_1V2: U$1.VOS
- removed net VREG: U$1.VIN
- new net DM: J1.D-
- new net DP: J1.D+
- new net IC21_SDA: J1.18
- new net IOB13B: J1.11
- new net IOB_0A: J1.22
- new net IOB_12A_G4_CDONE: J1.20
- new net IOB_24A: J1.7
- new net IOB_25B_G3: J1.17
- new net IOB_2A: J1.21
- new net IOB_3B_G6: J1.23
- new net IOB_9B: J1.16
- new net IOT47A: J1.4
- new net IOT_46B_G0: J1.8
- new net RGB0: J1.5
- new net RGB1: J1.10
- new net RGB2: J1.15
- new net SPI_CS: J1.13
- new net VBUS: J1.VB
- net BAT: no longer U$1.BAT
- net GND: now also J1.9, J1.GND, J1.S1, J1.S2, J1.S3, J1.S4; no longer J2.-, U$1.!CE!, U$1.EN1, U$1.GND, U$1.TD, U$1.VSEL, U$1.VSS
- net I2C1_SCL: now also J1.14
- net I2C2_SCL: now also J1.2
- net I2C2_SDA: now also J1.1
- net N$3: now also J1.24; no longer U$1.!PGOOD!
- net PV_VS: now also J5.P$8; no longer J2.+, J5.P$2
- net RTC_!INT!/RESET_B: now also J5.P$7; no longer J5.P$5
- net SPI_MISO: now also J1.12; no longer U$1.SO
- net SPI_MOSI: now also J1.6; no longer U$1.SI
- net SPI_SCK: now also J1.19; no longer U$1.SCK
- net SWD_CLK: now also J5.P$6; no longer J5.P$4
- net SWD_DIO: now also J5.P$5; no longer J5.P$3
- net USB_5V: now also J5.P$2
- net VCC: now also J1.3; no longer U$1.!RST!, U$1.VCC
- net VS1: now also J5.P$4; no longer U$1.1
- net VS2: now also J5.P$3
Other:
- note added: "14: VS2"
- note added: "5: VS1"
- note added: "Boost config resistors"
- note added: "Flash"
- note added: "Main boost circuit"
- note added: "Reset switch"
- note added: "SWD line set resistors"
- note added: "SWD socket"
- note added: "Supercaps"
- note added: "USB2"
- note removed: "14: VS_PRI"
- note removed: "5: VS_SEC"
- note removed: "FM ANT"
- note removed: "FT4222 pwr break"
- note removed: "PV cell JST socket"
- moved on the sheet: J4, J5, S1

Commit message: FPGA layout
Connections:
- removed net IC21_SDA: J1.18
- removed net IOB13B: J1.11
- removed net IOB_12A_G4_CDONE: J1.20
- removed net IOB_25B_G3: J1.17
- removed net IOT47A: J1.4
- removed net N$3: J1.24
- new net IOB_13B: J1.16
- new net IOT_47A: J1.2
- net GND: now also J1.18, J1.19; no longer J1.9
- net I2C1_SCL: now also J1.21; no longer J1.14
- net I2C1_SDA: now also J1.5
- net I2C2_SCL: now also J1.3; no longer J1.2
- net I2C2_SDA: now also J1.14; no longer J1.1
- net IOB_0A: now also J1.6; no longer J1.22
- net IOB_24A: now also J1.9; no longer J1.7
- net IOB_2A: now also J1.17; no longer J1.21
- net IOB_3B_G6: now also J1.11; no longer J1.23
- net IOB_9B: now also J1.22; no longer J1.16
- net IOT_46B_G0: now also J1.13; no longer J1.8
- net RGB0: now also J1.7; no longer J1.5
- net RGB1: now also J1.12; no longer J1.10
- net RGB2: now also J1.1; no longer J1.15
- net SPI_CS: now also J1.20; no longer J1.13
- net SPI_MISO: now also J1.10; no longer J1.12
- net SPI_MOSI: now also J1.15; no longer J1.6
- net SPI_SCK: now also J1.4; no longer J1.19
- net VCC: now also J1.8; no longer J1.3

Commit message: Top layout 70% complete
Parts:
- removed J5: DF40FC-20DP-0.4V(51), DF40FC-20DP-0.4V(51):DF40FC-20DP-0.4V(51)
- removed S2: CHS-04_SWITCH, CHS_SWITCH:CHS-04_SWITCH
- added J2: (no value), SparkFun-Connectors:JST_2MM_MALE
- added S3: CHS-02_SWITCH, CHS_SWITCH:CHS-02_SWITCH
Connections:
- removed net BOOST_EN: S2.1', S2.2'
- removed net BOOST_VBAT: S2.2
- removed net IOB_0A: J1.6
- removed net IOB_13B: J1.16
- removed net IOB_24A: J1.9
- removed net IOB_2A: J1.17
- removed net IOB_3B_G6: J1.11
- removed net IOB_9B: J1.22
- removed net IOT_46B_G0: J1.13
- removed net IOT_47A: J1.2
- removed net RGB0: J1.7
- removed net RGB1: J1.12
- removed net RGB2: J1.1
- removed net SPI_CS: J1.20
- removed net SPI_MISO: J1.10
- removed net SPI_MOSI: J1.15
- new net P10B: J2.P$10
- new net P11B: J2.P$11
- new net P12B: J2.P$12
- new net P13B: J2.P$13
- new net P14B: J2.P$14
- new net P15B: J2.P$15
- new net P16B: J2.P$16
- new net P17B: J2.P$17
- new net P18B: J2.P$18
- new net P19B: J2.P$19
- new net P1B: J2.P$1
- new net P20B: J2.P$20
- new net P2B: J2.P$2
- new net P3B: J2.P$3
- new net P4B: J2.P$4
- new net P5B: J2.P$5
- new net P6B: J2.P$6
- new net P7B: J2.P$7
- new net P8B: J2.P$8
- new net P9B: J2.P$9
- net BOOST_VOUT: now also S3.1; no longer S2.3
- net CHARGE_VOUT: now also S3.2; no longer S2.4
- net GND: now also J2.-, S3.B, S3.B'; no longer J1.18, J1.19, J5.P$1, S2.1
- net I2C1_SCL: no longer J1.21
- net I2C1_SDA: no longer J1.5
- net I2C2_SCL: no longer J1.3
- net I2C2_SDA: no longer J1.14
- net PTA1/RESET_B: now also S3.A, S3.A'
- net PV_VS: now also J2.+, J4.P$4; no longer J5.P$8
- net REG_VIN: now also S3.1', S3.2'; no longer S2.3', S2.4'
- net RTC_!INT!/RESET_B: no longer J5.P$7
- net SPI_SCK: no longer J1.4
- net SWD_CLK: no longer J5.P$6
- net SWD_DIO: no longer J5.P$5
- net USB_5V: no longer J5.P$2
- net VCC: no longer J1.8
- net VS1: no longer J4.P$4, J5.P$4
- net VS2: no longer J5.P$3
Other:
- note added: "2: Signal"
- note added: "3: GND"
- note removed: "2: GND"
- note removed: "3: Signal"
- note removed: "PV"
- moved on the sheet: J1

Commit message: Top layout removed USE SPI IC
Parts:
- added J5: DF40FC-20DP-0.4V(51), DF40FC-20DP-0.4V(51):DF40FC-20DP-0.4V(51)
- added U$1, U$2: MAX40200, MAX40200:MAX40200
Connections:
- new net AT45DB321F_SPI_CS: U$1.!CS!
- new net IN: U$1.IN
- new net N$1: U$1.ISET
- new net N$2: U$1.ILIM
- new net N$3: U$1.!PGOOD!
- new net N$4: U$1.!WP!, U$1.TS
- new net N$5: U$1.!CHG!
- new net N$8: U$1.TMR
- new net OUT: U$1.EN2, U$1.OUT
- new net REG_LOAD: U$2.IN
- new net SPI_MISO: U$1.SO
- new net SPI_MOSI: U$1.SI
- new net VCC_1V2: U$1.OUT
- new net VCC_QIIC: J3.VCC, U$1.IN
- new net VREG: U$1.IN
- net BAT: now also U$1.BAT
- net GND: now also U$1.!CE!, U$1.EN1, U$1.GND, U$1.TD, U$1.VSS, U$2.GND
- net SPI_SCK: now also U$1.SCK
- net VCC: now also U$1.!RST!, U$1.VCC
- net VS2: now also U$1.OUT, U$2.OUT; no longer J3.VCC
Other:
- note removed: "Sockets to break out lines"

Commit message: Start of bottom layer sensor routing
Parts:
- removed J5: DF40FC-20DP-0.4V(51), DF40FC-20DP-0.4V(51):DF40FC-20DP-0.4V(51)
Connections:
- net ADXL362_FT4222_SPI_CS renamed ADXL362_SPI_CS
- net ISL23415_SPI_CS/FT4222_GPIO3 renamed ISL23415_SPI_CS
- net PAN1326_!SHUTD renamed BGX13S_!RST
- net SI4705_!RST!/FT4222_GPIO2 renamed SI4705_!RST
- removed net P10A: J1.P$10
- removed net P10B: J2.P$10
- removed net P11A: J1.P$11
- removed net P11B: J2.P$11
- removed net P12A: J1.P$12
- removed net P12B: J2.P$12
- removed net P13A: J1.P$13
- removed net P13B: J2.P$13
- removed net P14A: J1.P$14
- removed net P14B: J2.P$14
- removed net P15A: J1.P$15
- removed net P15B: J2.P$15
- removed net P16A: J1.P$16
- removed net P16B: J2.P$16
- removed net P17A: J1.P$17
- removed net P17B: J2.P$17
- removed net P18A: J1.P$18
- removed net P18B: J2.P$18
- removed net P19A: J1.P$19
- removed net P19B: J2.P$19
- removed net P1A: J1.P$1
- removed net P1B: J2.P$1
- removed net P20A: J1.P$20
- removed net P20B: J2.P$20
- removed net P2A: J1.P$2
- removed net P2B: J2.P$2
- removed net P3A: J1.P$3
- removed net P3B: J2.P$3
- removed net P4A: J1.P$4
- removed net P4B: J2.P$4
- removed net P5A: J1.P$5
- removed net P5B: J2.P$5
- removed net P6A: J1.P$6
- removed net P6B: J2.P$6
- removed net P7A: J1.P$7
- removed net P7B: J2.P$7
- removed net P8A: J1.P$8
- removed net P8B: J2.P$8
- removed net P9A: J1.P$9
- removed net P9B: J2.P$9
Other:
- note removed: "DF40 Sockets"
- note removed: "I2C Address: 0x3A (ADDR0 -> GND)"
- moved on the sheet: J1, J2, J4, S3

Commit message: Bottom sensor placement
Other:
- note added: "Digipots"

Commit message: All chips routed
Parts:
- removed FD4: FIDUCIAL1X2, SparkFun-Aesthetics:FIDUCIAL1X2
- J2: value (none) -> QIIC connector; device SparkFun-Connectors:JST_2MM_MALE -> SparkX:I2C_STANDARDJS-1MM
Connections:
- removed net ADXL362_SPI_CS: J4.P$18
- net BGX13S_!RST: now also J4.P$7; no longer J4.P$20
- net GND: now also J2.GND, J4.P$20; no longer J2.-, J4.P$1
- net I2C0_SCL/UART_TX: now also J4.P$5; no longer J3.SCL, J4.P$11
- net I2C0_SDA/UART_RX: now also J4.P$6; no longer J3.SDA, J4.P$12
- net I2C1_SCL: now also J2.SCL, J4.P$1; no longer J4.P$13
- net I2C1_SDA: now also J2.SDA, J4.P$2; no longer J4.P$14
- net I2C2_SCL: now also J3.SCL, J4.P$3; no longer J4.P$15
- net I2C2_SDA: now also J3.SDA, J4.P$4; no longer J4.P$16
- net ISL23415_SPI_CS: now also J4.P$16; no longer J4.P$17
- net PV_VS: now also J4.P$15; no longer J2.+, J4.P$4
- net RTC_!INT!/RESET_B: now also J4.P$10; no longer J4.P$7
- net SI4705_!RST: now also J4.P$17; no longer J4.P$19
- net SPI_MISO/UART_RTS: now also J4.P$12; no longer J4.P$9
- net SPI_MOSI/UART_CTS: now also J4.P$13; no longer J4.P$10
- net SPI_SCK: now also J4.P$11; no longer J4.P$8
- net SWD_CLK: now also J4.P$9; no longer J4.P$6
- net SWD_DIO: now also J4.P$8; no longer J4.P$5
- net USB_5V: now also J4.P$14; no longer J4.P$2
- net VCC_QIIC: now also J2.VCC
- net VS1: now also J4.P$18
- net VS2: now also J4.P$19; no longer J4.P$3
Other:
- note added: "19/9/19"
- note added: "Bluetooth"
- note added: "Consolidated breakout boards Removed FT4222 USB interface FPGA driven using LDO Changed Bluetooth module to BGX13S Added digipots for each sensor i2c bus Added QIIC connects for each i2c bus Added ideal diodes to protect regulator from QIIC supply voltage Removed one DF40 header Removed RTC battery Removed Grideye sensor"
- note added: "DIGIPOT"
- note added: "MAIN"
- note added: "PCB"
- note added: "SENSORS2"
- moved on the sheet: S1
