File: revB/cad/eagle/warp-revC.sch (EAGLE design)
At the start: 12 parts, among them J2 QIIC connector, J3 QIIC connector, J4 DF40FC-20DP-0.4V(51)

Commit message: Corrected DRC errors with layout and completed silkscreen
Parts:
- removed FD5: FIDUCIAL1X2, SparkFun-Aesthetics:FIDUCIAL1X2
- removed S3: CHS-02_SWITCH, CHS_SWITCH:CHS-02_SWITCH
- removed U$2: MAX40200, MAX40200:MAX40200
- added FD4: FIDUCIAL1X2, SparkFun-Aesthetics:FIDUCIAL1X2
- added J5: CORTEX_DEBUG_SMD, SparkFun-Connectors:CORTEX_DEBUG_SMD
- added S2: CHS-02_SWITCH, CHS_SWITCH:CHS-02_SWITCH
- added U1: MAX40200, MAX40200:MAX40200
- renumbered U$1 to U2
Connections:
- net PV_VS renamed PV_VIN
- removed net BOOST_VOUT: S3.1
- removed net DM: J1.D-
- removed net DP: J1.D+
- new net !INT: U1.!INT!
- new net !RESET: U1.!RESET
- new net ADXL362_SPI_CS: U1.!CS
- new net BQ24230_OUT: U1.EN2, U1.OUT, U2.IN
- new net CAP: U2.CAP
- new net CRESET_B: U2.CRESET_B
- new net CTRL: U1.CTRL
- new net DCP_RW1: U1.RW
- new net DCP_RW3: U2.RW
- new net EXTAL0: U1.PTA3/EXTAL0
- new net I2C_SCL: U1.SCL, U2.I2C_SCL/SPI_SPC, U2.SCX
- new net I2C_SCL/LPUART0_TX: U1.PTB3/IRQ_10
- new net I2C_SDA: U1.SDA, U2.I2C_SDA/SPI_SDI/SPI3_SDO, U2.SDX
- new net I2C_SDA/LPUART0_RX: U1.PTB4/IRQ_11
- new net ICE40_VCC_PLL: U2.IOB_24A, U2.VCCPLL
- new net LBOOST: U1.LBOOST
- new net LBUCK: U1.LBUCK
- new net LOAD: U1.LOAD
- new net OK_HYST: U1.OK_HYST
- new net OK_PROG: U1.OK_PROG
- new net PTA12: U1.PTA12/IRQ_13/LPTMR0_ALT2
- new net PTA5: U1.PTA5/RTC_CLK_IN
- new net PTA8: U1.PTA8
- new net PTB1: U1.PTB1/IRQ_6/ADC0_SE8/CMP0_IN3
- new net PTB10: U1.PTB10
- new net PTB11: U1.PTB11
- new net PTB13/CLKOUT32K: U1.PTB13/CLKOUT32K
- new net PTB2: U1.PTB2/IRQ_7
- new net PTB5: U1.PTB5/IRQ_12
- new net PTB6: U1.PTB6/IRQ_2/LPTMR0_ALT3
- new net PTB7: U1.PTB7/IRQ_3
- new net PV_VOUT: S2.1
- new net SPI_CS: U1.CS, U2.CS, U2.IOB_35B_SPI_SS
- new net SW: U1.SW
- new net UART_CTS: U1.UART_CTS
- new net UART_RTS: U1.UART_RTS
- new net UART_RX: U1.UART_RX
- new net UART_TX: U1.UART_TX
- new net VBAT: U1.VBAT
- new net VBAT_OV: U1.VBAT_OV
- new net VIN: U1.EN, U1.VIN, U1.VIN_DC
- new net VOUT: U1.VOUT
- new net VOUT_SET: U1.VOUT_SET
- new net VRDIV: U1.VRDIV
- new net VREF_SAMP: U1.VREF_SAMP
- new net VSEL1: U1.VSEL1
- new net VSEL2: U1.VSEL2
- new net VSEL3: U1.VSEL3
- new net VSEL4: U1.VSEL4
- new net VSTOR: U1.VOC_SAMP, U1.VOUT_EN, U1.VSTOR
- new net XTAL0: U1.PTA4/XTAL0
- net AT45DB321F_SPI_CS: now also U1.PTA9
- net BAT: now also U1.BAT; no longer U2.BAT
- net CHARGE_VOUT: now also S2.2; no longer S3.2
- net GND: now also J5.GND@3, J5.GND@5, S1.B, S1.B', U1.!CE!, U1.!EN, U1.ANT_GND, U1.CLKOE, U1.EN1, U1.GND, U1.GND@10, U1.GND@12, U1.GND@13, U1.GND@16, U1.GND@5, U1.NC17, U1.NC9, U1.PAD, U1.SA0, U1.SHIELD, U1.TD, U1.VGND, U1.VSS, U1.VSS1, U1.VSS15, U2.CSB3, U2.GND@12, U2.GND@13, U2.GNDA, U2.GNDIO, U2.I2C_SA0/SPI_SDO, U2.RESERVED@10, U2.RESERVED@11, U2.RESERVED@15, U2.RESERVED@9, U2.SDO1, U2.SDO2, U2.VGND; no longer J1.GND, J1.GND@3, J1.GND@5, J1.S1, J1.S2, J1.S3, J1.S4, S3.B, S3.B', U$2.GND, U2.!CE!, U2.EN1, U2.TD, U2.VSS
- net I2C1_SCL: now also J3.SCL, U2.IOT_47A; no longer J2.SCL
- net I2C1_SDA: now also J3.SDA, U2.IOB_11B_G5; no longer J2.SDA
- net I2C2_SCL: now also J2.SCL, U2.IOT_37A; no longer J3.SCL
- net I2C2_SDA: now also J2.SDA, U2.IOT_36B; no longer J3.SDA
- net IN: now also U1.IN; no longer U2.IN
- net N$1: now also U1.BYP, U1.ISET, U1.LFXTAL_N; no longer U2.ISET
- net N$2: now also U1.ILIM, U1.LFXTAL_P; no longer U2.ILIM
- net N$3: now also U1.!PGOOD!, U1.ANTENNA, U1.EVI, U1.RF; no longer U2.!PGOOD!
- net N$4: now also U1.TS; no longer U2.TS
- net N$5: now also U1.!CHG!; no longer U2.!CHG!
- net N$8: now also U1.TMR; no longer U2.TMR
- net OUT: no longer U2.EN2
- net PTA0/SWD_CLK: now also U1.PTA0/IRQ_0/LLWU_P7; no longer J1.SWDCLK/TCK
- net PTA1/RESET_B: now also S1.A, S1.A', U1.PTA1/IRQ1/LPTMR0_ALT1; no longer J1.!RESET, S3.A, S3.A'
- net PTA2/SWD_DIO: now also U1.PTA2; no longer J1.SWDIO/TMS
- net REG_LOAD: now also U1.IN; no longer U$2.IN
- net REG_VIN: now also S2.1', S2.2'; no longer S3.1', S3.2'
- net RTC_!INT!/RESET_B: now also J5.!RESET
- net SPI_MISO: now also U1.MISO, U1.PTA6, U1.SDO, U2.IOB_32A_SPI_SO, U2.SDO
- net SPI_MOSI: now also U1.MOSI, U1.PTA7/IRQ_4, U1.SDI, U2.IOB_33B_SPI_SI, U2.SDI
- net SPI_SCK: now also U1.PTB0/IRQ_5/LLWU_P4, U1.SCK, U1.SCLK, U2.IOB_34A_SPI_SCK
- net SWD_CLK: now also J5.SWDCLK/TCK
- net SWD_DIO: now also J5.SWDIO/TMS
- net VBUS: now also U1.VBUS; no longer J1.VB
- net VCC: now also U1.IOVDD, U1.RL, U1.VBATT, U1.VCC, U1.VDD, U1.VDDIO, U1.VLOGIC, U1.VS, U2.I2C_VS_SPI_MODE_SELECT, U2.PS, U2.RL, U2.SPI_VCCIO1, U2.VCCIO_0, U2.VCCIO_2, U2.VDD, U2.VDDIO, U2.VDD_IO, U2.VLOGIC, U2.VPP_2V5; no longer J1.VCC
- net VCC_1V2: now also U1.OUT, U2.VCC; no longer U2.OUT
- net VREG: now also U1.IN; no longer U2.IN
- net VS1: now also J5.VCC
- net VS2: now also U1.OUT; no longer U$2.OUT
Other:
- note added: "2: GND / WLP breakout"
- note added: "7/10/19"
- note added: "Swapped micro USB part"
- note removed: "2: Signal"
- note removed: "I2C"
- note removed: "PWR"
- note removed: "SPI"
- note removed: "SWD"
- note removed: "UART"
- note removed: "USB supply"
- moved on the sheet: J2, J3, S1
